Commit message: Fixed model typ

File: t_frog_description/urdf/t_frog.xacro (robot description, xacro)
@@ -15,167 +15,139 @@
   <xacro:include filename="$(find t_frog_description)/urdf/materials.xacro" />
   <!-- Used for fixing robot to Gazebo 'base_link' -->
+  <!--
   <link name="world"/>
   <joint name="fixed" type="fixed">
     <parent link="world"/>
-    <child link="link1"/>
+    <child link="base_link"/>
   </joint>
+  -->
   <!-- Base Link -->
-  <link name="link1">
+  <link name="base_link">
     <collision>
-      <origin xyz="0 0 ${height1/2}" rpy="0 0 0"/>
+      <origin xyz="0 0 .1" rpy="0 0 0"/>
       <geometry>
-	<box size="${width} ${width} ${height1}"/>
+	<box size=".4 .2 .1"/>
       </geometry>
     </collision>
     <visual>
-      <origin xyz="0 0 ${height1/2}" rpy="0 0 0"/>
+      <origin xyz="0 0 .1" rpy="0 0 0"/>
       <geometry>
-	<box size="${width} ${width} ${height1}"/>
+	<box size=".4 .2 .1"/>
       </geometry>
       <material name="orange"/>
     </visual>
     <inertial>
-      <origin xyz="0 0 ${height1/2}" rpy="0 0 0"/>
-      <mass value="1"/>
-      <inertia
-	  ixx="1.0" ixy="0.0" ixz="0.0"
-	  iyy="1.0" iyz="0.0"
-	  izz="1.0"/>
+       <mass value="1e-5" />
+       <origin xyz="0 0 .1 " rpy="0 0 0"/>
+       <inertia ixx="1e-6" ixy="0" ixz="0" iyy="1e-6" iyz="0" izz="1e-6" />
     </inertial>
   </link>
-  <joint name="joint1" type="continuous">
-    <parent link="link1"/>
-    <child link="link2"/>
-    <origin xyz="0 ${width} ${height1 - axel_offset}" rpy="0 0 0"/>
-    <axis xyz="0 1 0"/>
-    <dynamics damping="0.7"/>
-  </joint>
-  <!-- Middle Link -->
-  <link name="link2">
-    <collision>
-      <origin xyz="0 0 ${height2/2 - axel_offset}" rpy="0 0 0"/>
+  <link name="left_wheel">
+    <collision name="collision">
+      <origin xyz=".1 0.13 .1" rpy="0 1.5707 1.5707"/>
       <geometry>
-	<box size="${width} ${width} ${height2}"/>
+         <cylinder  length="0.05" radius="0.1"/>
       </geometry>
     </collision>
-    <visual>
-      <origin xyz="0 0 ${height2/2 - axel_offset}" rpy="0 0 0"/>
+    <visual name="visual">
+      <origin xyz=".1 0.13 .1" rpy="0 1.5707 1.5707"/>
       <geometry>
-	<box size="${width} ${width} ${height2}"/>
-      </geometry>
-      <material name="black"/>
-    </visual>
-    <inertial>
-      <origin xyz="0 0 ${height2/2 - axel_offset}" rpy="0 0 0"/>
-      <mass value="1"/>
-      <inertia
-	  ixx="1.0" ixy="0.0" ixz="0.0"
-	  iyy="1.0" iyz="0.0"
-	  izz="1.0"/>
-    </inertial>
-  </link>
-  <joint name="joint2" type="continuous">
-    <parent link="link2"/>
-    <child link="link3"/>
-    <origin xyz="0 ${width} ${height2 - axel_offset*2}" rpy="0 0 0"/>
-    <axis xyz="0 1 0"/>
-    <dynamics damping="0.7"/>
-  </joint>
-  <!-- Top Link -->
-  <link name="link3">
-    <collision>
-      <origin xyz="0 0 ${height3/2 - axel_offset}" rpy="0 0 0"/>
-      <geometry>
-	<box size="${width} ${width} ${height3}"/>
-      </geometry>
-    </collision>
-    <visual>
-      <origin xyz="0 0 ${height3/2 - axel_offset}" rpy="0 0 0"/>
-      <geometry>
-	<box size="${width} ${width} ${height3}"/>
-      </geometry>
-      <material name="orange"/>
-    </visual>
-    <inertial>
-      <origin xyz="0 0 ${height3/2 - axel_offset}" rpy="0 0 0"/>
-      <mass value="1"/>
-      <inertia
-	  ixx="1.0" ixy="0.0" ixz="0.0"
-	  iyy="1.0" iyz="0.0"
-	  izz="1.0"/>
-    </inertial>
-  </link>
-  <joint name="hokuyo_joint" type="fixed">
-    <axis xyz="0 1 0" />
-    <origin xyz="0 0 ${height3 - axel_offset/2}" rpy="0 0 0"/>
-    <parent link="link3"/>
-    <child link="hokuyo_link"/>
-  </joint>
-  <!-- Hokuyo Laser -->
-  <link name="hokuyo_link">
-    <collision>
-      <origin xyz="0 0 0" rpy="0 0 0"/>
-      <geometry>
-	<box size="0.1 0.1 0.1"/>
-      </geometry>
-    </collision>
-    <visual>
-      <origin xyz="0 0 0" rpy="0 0 0"/>
-      <geometry>
-        <mesh filename="package://t_frog_description/meshes/hokuyo.dae"/>
+        <cylinder  length="0.05" radius="0.1"/>
       </geometry>
     </visual>
     <inertial>
       <mass value="1e-5" />
-      <origin xyz="0 0 0" rpy="0 0 0"/>
+      <origin xyz=".1 0.13 .1"/>
       <inertia ixx="1e-6" ixy="0" ixz="0" iyy="1e-6" iyz="0" izz="1e-6" />
     </inertial>
   </link>
-  <joint name="camera_joint" type="fixed">
-    <axis xyz="0 1 0" />
-    <origin xyz="${camera_link} 0 ${height3 - axel_offset*2}" rpy="0 0 0"/>
-    <parent link="link3"/>
-    <child link="camera_link"/>
+  <joint type="revolute" name="left_wheel_hinge">
+    <origin xyz="0 0.03 0" rpy="0 0 0"/>
+    <child link="left_wheel">left_wheel</child>
+    <parent link="base_link">base_link</parent>
+    <axis xyz="0 1 0"/>
+    <limit effort="30" velocity="1.0"  lower="-100" upper="100" />
   </joint>
-  <!-- Camera -->
-  <link name="camera_link">
+  <link name="right_wheel">
+    <collision name="collision">
+      <origin xyz="0.1 -0.13 0.1" rpy="0 1.5707 1.5707"/>
+      <geometry>
+         <cylinder  length="0.05" radius="0.1"/>
+      </geometry>
+    </collision>
+    <visual name="visual">
+      <origin xyz="0.1 -0.13 0.1" rpy="0 1.5707 1.5707"/>
+      <geometry>
+        <cylinder  length="0.05" radius="0.1"/>
+      </geometry>
+    </visual>
+    <inertial>
+      <mass value="1e-5" />
+      <origin xyz="0.1 -0.13 0.1"/>
+      <inertia ixx="1e-6" ixy="0" ixz="0" iyy="1e-6" iyz="0" izz="1e-6" />
+    </inertial>
+  </link>
+  <joint type="revolute" name="right_wheel_hinge">
+    <origin xyz="0 -0.03 0" rpy="0 0 0"/>
+    <child link="right_wheel">right_wheel</child>
+    <parent link="base_link">base_link</parent>
+    <axis xyz="0 1 0"/>
+    <limit effort="30" velocity="1.0"  lower="-100" upper="100" />
+  </joint>
+<!--
+  <joint name="left_wheel_hinge" type="revolute">
+    <parent link="chassis"/>
+    <child link="left_wheel"/>
+    <origin xyz="0 0 -0.03" rpy="0 0 0"/>
+    <axis xyz="0 1 0"/>
+  </joint>
+<link name="left_wheel">
     <collision>
-      <origin xyz="0 0 0" rpy="0 0 0"/>
+      <origin xyz="0.1 0.13 0.1" rpy="0 1.5707 1.5707"/>
       <geometry>
-	<box size="${camera_link} ${camera_link} ${camera_link}"/>
+        <cylinder>
+	  <radius>.1</radius>
+	  <length>.05</length>
+	</cylinder>
       </geometry>
     </collision>
     <visual>
-      <origin xyz="0 0 0" rpy="0 0 0"/>
+      <origin xyz="0.1 0.13 0.1" rpy="0 1.5707 1.5707"/>
       <geometry>
-	<box size="${camera_link} ${camera_link} ${camera_link}"/>
+        <cylinder>
+	  <radius>.1</radius>
+	  <length>.05</length>
+	</cylinder>
       </geometry>
-      <material name="red"/>
+      <material name="orange"/>
     </visual>
-    <inertial>
-      <mass value="1e-5" />
-      <origin xyz="0 0 0" rpy="0 0 0"/>
-      <inertia ixx="1e-6" ixy="0" ixz="0" iyy="1e-6" iyz="0" izz="1e-6" />
-    </inertial>
   </link>
-  <transmission name="tran1">
-    <type>transmission_interface/SimpleTransmission</type>
-    <joint name="joint1">
-      <hardwareInterface>EffortJointInterface</hardwareInterface>
-    </joint>
-  <actuator name="motor1">
-      <hardwareInterface>EffortJointInterface</hardwareInterface>
-      <mechanicalReduction>1</mechanicalReduction>
-    </actuator>
-  </transmission>
-  <transmission name="tran2">
-    <type>transmission_interface/SimpleTransmission</type>
-    <joint name="joint2">
-      <hardwareInterface>EffortJointInterface</hardwareInterface>
-    </joint>
-  <actuator name="motor2">
-      <hardwareInterface>EffortJointInterface</hardwareInterface>
-      <mechanicalReduction>1</mechanicalReduction>
-    </actuator>
-  </transmission>
+  <joint name="right_wheel_hinge" type="revolute">
+    <parent link="chassis"/>
+    <child link="right_wheel"/>
+    <origin xyz="0 0 0.03" rpy="0 0 0"/>
+    <axis xyz="0 1 0"/>
+  </joint>
+  <link name="right_wheel">
+    <collision>
+      <origin xyz="0.1 -0.13 0.1" rpy="0 1.5707 1.5707"/>
+      <geometry>
+        <cylinder>
+	  <radius>.1</radius>
+	  <length>.05</length>
+	</cylinder>
+      </geometry>
+    </collision>
+    <visual>
+      <origin xyz="0.1 -0.13 0.1" rpy="0 1.5707 1.5707"/>
+      <geometry>
+        <cylinder>
+	  <radius>.1</radius>
+	  <length>.05</length>
+	</cylinder>
+      </geometry>
+      <material name="orange"/>
+    </visual>
+  </link>
+-->
 </robot>

Commit message: Fix a position of the rotation center

File: t_frog_description/urdf/t_frog.xacro (robot description, xacro)
@@ -45,5 +45,5 @@
   <link name="left_wheel">
     <collision name="collision">
-      <origin xyz=".1 0.13 .1" rpy="0 1.5707 1.5707"/>
+      <origin xyz="0 0.03 0" rpy="0 1.5707 1.5707"/>
       <geometry>
          <cylinder  length="0.05" radius="0.1"/>
@@ -51,5 +51,5 @@
     </collision>
     <visual name="visual">
-      <origin xyz=".1 0.13 .1" rpy="0 1.5707 1.5707"/>
+      <origin xyz="0 0.03 0" rpy="0 1.5707 1.5707"/>
       <geometry>
         <cylinder  length="0.05" radius="0.1"/>
@@ -58,10 +58,10 @@
     <inertial>
       <mass value="1e-5" />
-      <origin xyz=".1 0.13 .1"/>
+      <origin xyz="0 0.03 0"/>
       <inertia ixx="1e-6" ixy="0" ixz="0" iyy="1e-6" iyz="0" izz="1e-6" />
     </inertial>
   </link>
   <joint type="revolute" name="left_wheel_hinge">
-    <origin xyz="0 0.03 0" rpy="0 0 0"/>
+    <origin xyz="0.1 0.13 0.1" rpy="0 0 0"/>
     <child link="left_wheel">left_wheel</child>
     <parent link="base_link">base_link</parent>
@@ -71,5 +71,5 @@
   <link name="right_wheel">
     <collision name="collision">
-      <origin xyz="0.1 -0.13 0.1" rpy="0 1.5707 1.5707"/>
+      <origin xyz="0 -0.03 0" rpy="0 1.5707 1.5707"/>
       <geometry>
          <cylinder  length="0.05" radius="0.1"/>
@@ -77,5 +77,5 @@
     </collision>
     <visual name="visual">
-      <origin xyz="0.1 -0.13 0.1" rpy="0 1.5707 1.5707"/>
+      <origin xyz="0 -0.03 0" rpy="0 1.5707 1.5707"/>
       <geometry>
         <cylinder  length="0.05" radius="0.1"/>
@@ -84,10 +84,10 @@
     <inertial>
       <mass value="1e-5" />
-      <origin xyz="0.1 -0.13 0.1"/>
+      <origin xyz="0 -0.03 0"/>
       <inertia ixx="1e-6" ixy="0" ixz="0" iyy="1e-6" iyz="0" izz="1e-6" />
     </inertial>
   </link>
   <joint type="revolute" name="right_wheel_hinge">
-    <origin xyz="0 -0.03 0" rpy="0 0 0"/>
+    <origin xyz="0.1 -0.13 0.1" rpy="0 0 0"/>
     <child link="right_wheel">right_wheel</child>
     <parent link="base_link">base_link</parent>
@@ -95,59 +95,3 @@
     <limit effort="30" velocity="1.0"  lower="-100" upper="100" />
   </joint>
-<!--
-  <joint name="left_wheel_hinge" type="revolute">
-    <parent link="chassis"/>
-    <child link="left_wheel"/>
-    <origin xyz="0 0 -0.03" rpy="0 0 0"/>
-    <axis xyz="0 1 0"/>
-  </joint>
-<link name="left_wheel">
-    <collision>
-      <origin xyz="0.1 0.13 0.1" rpy="0 1.5707 1.5707"/>
-      <geometry>
-        <cylinder>
-	  <radius>.1</radius>
-	  <length>.05</length>
-	</cylinder>
-      </geometry>
-    </collision>
-    <visual>
-      <origin xyz="0.1 0.13 0.1" rpy="0 1.5707 1.5707"/>
-      <geometry>
-        <cylinder>
-	  <radius>.1</radius>
-	  <length>.05</length>
-	</cylinder>
-      </geometry>
-      <material name="orange"/>
-    </visual>
-  </link>
-  <joint name="right_wheel_hinge" type="revolute">
-    <parent link="chassis"/>
-    <child link="right_wheel"/>
-    <origin xyz="0 0 0.03" rpy="0 0 0"/>
-    <axis xyz="0 1 0"/>
-  </joint>
-  <link name="right_wheel">
-    <collision>
-      <origin xyz="0.1 -0.13 0.1" rpy="0 1.5707 1.5707"/>
-      <geometry>
-        <cylinder>
-	  <radius>.1</radius>
-	  <length>.05</length>
-	</cylinder>
-      </geometry>
-    </collision>
-    <visual>
-      <origin xyz="0.1 -0.13 0.1" rpy="0 1.5707 1.5707"/>
-      <geometry>
-        <cylinder>
-	  <radius>.1</radius>
-	  <length>.05</length>
-	</cylinder>
-      </geometry>
-      <material name="orange"/>
-    </visual>
-  </link>
--->
 </robot>

Commit message: Added transmission tabs

File: t_frog_description/urdf/t_frog.xacro (robot description, xacro)
@@ -17,5 +17,5 @@
   <!--
   <link name="world"/>
-  <joint name="fixed" type="fixed">
+  <joint name="continuous" type="continuous">
     <parent link="world"/>
     <child link="base_link"/>
@@ -95,3 +95,23 @@
     <limit effort="30" velocity="1.0"  lower="-100" upper="100" />
   </joint>
+  <transmission name="tran1">
+    <type>transmission_interface/SimpleTransmission</type>
+    <joint name="left_wheel_hinge">
+      <hardwareInterface>VelocityJointInterface</hardwareInterface>
+    </joint>
+  <actuator name="left_motor">
+      <hardwareInterface>VelocityJointInterface</hardwareInterface>
+      <mechanicalReduction>1</mechanicalReduction>
+    </actuator>
+  </transmission>
+  <transmission name="tran2">
+    <type>transmission_interface/SimpleTransmission</type>
+    <joint name="right_wheel_hinge">
+      <hardwareInterface>VelocityJointInterface</hardwareInterface>
+    </joint>
+  <actuator name="right_motor">
+      <hardwareInterface>VelocityJointInterface</hardwareInterface>
+      <mechanicalReduction>1</mechanicalReduction>
+    </actuator>
+  </transmission>
 </robot>

Commit message: Added an caster joint

File: t_frog_description/urdf/t_frog.xacro (robot description, xacro)
@@ -34,4 +34,27 @@
       <geometry>
 	<box size=".4 .2 .1"/>
+      </geometry>
+      <material name="orange"/>
+    </visual>
+    <collision>
+      <origin xyz="-0.15 0 0.03" rpy="0 0 0"/>
+      <geometry>
+	<sphere radius="0.02"/>
+      </geometry>
+      <surface>
+        <friction>
+          <ode>
+	    <mu>0</mu>
+	    <mu2>0</mu2>
+	    <slip1>1.0</slip1>
+	    <slip2>1.0</slip2>
+	  </ode>
+        </friction>
+      </surface>
+    </collision>
+    <visual>
+      <origin xyz="-0.15 0 0.03" rpy="0 0 0"/>
+      <geometry>
+	<sphere radius="0.02"/>
       </geometry>
       <material name="orange"/>

Commit message: Added sensor links

File: t_frog_description/urdf/t_frog.xacro (robot description, xacro)
@@ -118,4 +118,55 @@
     <limit effort="30" velocity="1.0"  lower="-100" upper="100" />
   </joint>
+  <joint name="hokuyo_joint" type="fixed">
+    <axis xyz="0 1 0"/>
+    <origin xyz="0 0 0.175" rpy="0 0 0"/>
+    <parent link="base_link"/>
+    <child link="hokuyo_link"/>
+  </joint>
+  <link name="hokuyo_link">
+    <collision>
+      <origin xyz="0 0 0" rpy="0 0 0"/>
+      <geometry>
+        <box size="0.1 0.1 0.1"/>
+      </geometry>
+    </collision>
+    <visual>
+      <origin xyz="0 0 0" rpy="0 0 0"/>
+      <geometry>
+        <mesh filename="package://t_frog_description/meshes/hokuyo.dae"/>
+      </geometry>
+    </visual>
+    <inertial>
+      <mass value="1e-5"/>
+      <origin xyz="0 0 0" rpy="0 0 0"/>
+      <inertia ixx="1e-6" ixy="0" ixz="0" iyy="1e-6" iyz="0" izz="1e-6"/>
+    </inertial>
+  </link>
+  <joint name="camera_joint" type="fixed">
+    <axis xyz="0 1 0" />
+    <origin xyz="0.2 0 0.175" rpy="0 0 0"/>
+    <parent link="base_link"/>
+    <child link="camera_link"/>
+  </joint>
+  <link name="camera_link">
+    <collision>
+      <origin xyz="0 0 0" rpy="0 0 0"/>
+      <geometry>
+        <box size="${camera_link} ${camera_link} ${camera_link}"/>
+      </geometry>
+    </collision>
+    <visual>
+      <origin xyz="0 0 0" rpy="0 0 0"/>
+      <geometry>
+        <box size="${camera_link} ${camera_link} ${camera_link}"/>
+      </geometry>
+      <material name="red"/>
+    </visual>
+    <inertial>
+      <mass value="1e-5" />
+      <origin xyz="0 0 0" rpy="0 0 0"/>
+      <inertia ixx="1e-6" ixy="0" ixz="0" iyy="1e-6" iyz="0" izz="1e-6" />
+    </inertial>
+  </link>
   <transmission name="tran1">
     <type>transmission_interface/SimpleTransmission</type>

Commit message: Defined const data

File: t_frog_description/urdf/t_frog.xacro (robot description, xacro)
@@ -8,6 +8,7 @@
   <xacro:property name="height2" value="1" /> <!-- Link 2 -->
   <xacro:property name="height3" value="1" /> <!-- Link 3 -->
-  <xacro:property name="camera_link" value="0.05" /> <!-- Size of square 'camera' box -->
-  <xacro:property name="axel_offset" value="0.05" /> <!-- Space btw top of beam and the each joint -->
+  <xacro:property name="camera_link" value="0.05"/> <!-- Size of square 'camera' box -->
+  <xacro:property name="hokuyo_link" value="0.1" /> <!-- Size of square 'hokuyo' box -->
+  <xacro:property name="axel_offset" value="0.05"/> <!-- Space btw top of beam and the each joint -->
   <!-- Import all Gazebo-customization elements, including Gazebo colors -->
   <xacro:include filename="$(find t_frog_description)/urdf/t_frog.gazebo" />
@@ -128,5 +129,5 @@
       <origin xyz="0 0 0" rpy="0 0 0"/>
       <geometry>
-        <box size="0.1 0.1 0.1"/>
+        <box size="${hokuyo_link} ${hokuyo_link} ${hokuyo_link}"/>
       </geometry>
     </collision>
