Commit message: icart_middleのurdf完成(仮)

File: orne_description/urdf/icart_middle.xacro (robot description, xacro)
@@ -6,5 +6,5 @@
   <!-- Import Rviz colors -->
   <xacro:include filename="$(find icart_mini_description)/urdf/materials.xacro" />
-  <xacro:include filename="$(find icart_mini_description)/urdf/icart_mini.gazebo"/>
+  <xacro:include filename="$(find orne_description)/urdf/icart_middle.gazebo"/>
   <!-- Base Link -->
   <link name="base_link">
@@ -12,5 +12,5 @@
       <origin xyz="0 0 0.1" rpy="0 0 0"/>
       <geometry>
-	<box size=".485 .43 .15"/>
+	<box size=".462 .50 .134"/>
       </geometry>
     </collision>
@@ -18,10 +18,23 @@
       <origin xyz="0 0 0.1" rpy="0 0 0"/>
       <geometry>
-	<box size=".485 .43 .15"/>
+	<box size=".462 .50 .134"/>
+      </geometry>
+      <material name="orange"/>
+    </visual>
+    <collision>
+      <origin xyz="-0.095 0 0.305" rpy="0 0 0"/>
+      <geometry>
+	<box size=".276 .50 .342"/>
+      </geometry>
+    </collision>
+    <visual>
+      <origin xyz="-0.095 0 0.305" rpy="0 0 0"/>
+      <geometry>
+	<box size=".276 .50 .342"/>
       </geometry>
       <material name="orange"/>
     </visual>
     <collision name="collision">
-      <origin xyz="-0.175 0.0 0.05" rpy="0 1.5707 1.5707"/>
+      <origin xyz="-0.231 -0.141 0.05" rpy="0 1.5707 1.5707"/>
       <geometry>
         <cylinder  length="0.03" radius="0.04625"/>
@@ -29,5 +42,5 @@
     </collision>
     <visual name="visual">
-      <origin xyz="-0.175 0.0 0.05" rpy="0 1.5707 1.5707"/>
+      <origin xyz="-0.231 -0.141 0.05" rpy="0 1.5707 1.5707"/>
       <geometry>
         <cylinder  length="0.03" radius="0.04625"/>
@@ -35,9 +48,15 @@
     </visual>
     <collision name="collision">
-      <origin xyz="0.175 0.0 0.05" rpy="0 1.5707 1.5707"/>
+      <origin xyz="-0.231 0.141 0.05" rpy="0 1.5707 1.5707"/>
       <geometry>
         <cylinder  length="0.03" radius="0.04625"/>
       </geometry>
     </collision>
+    <visual name="visual">
+      <origin xyz="-0.231 0.141 0.05" rpy="0 1.5707 1.5707"/>
+      <geometry>
+        <cylinder  length="0.03" radius="0.04625"/>
+      </geometry>
+    </visual>
     <inertial>
        <mass value="20" />
@@ -50,10 +69,10 @@
       <origin xyz="0 0.0 0" rpy="0 1.5707 1.5707"/>
       <geometry>
-        <cylinder  length="0.03" radius="0.0725"/>
+        <cylinder  length="0.03" radius="0.151"/>
       </geometry>
     </visual>
   </link>
   <joint type="fixed" name="visual_left_wheel_hinge">
-    <origin xyz="0.15 0.15 0.075" rpy="0 0 0"/>
+    <origin xyz="0.06 0.288 0.1518" rpy="0 0 0"/>
     <child link="visual_left_wheel">visual_left_wheel</child>
     <parent link="base_link">base_link</parent>
@@ -64,5 +83,5 @@
       <origin xyz="0 0.0 0" rpy="0 1.5707 1.5707"/>
       <geometry>
-         <cylinder  length="0.03" radius="0.0725"/>
+         <cylinder  length="0.03" radius="0.151"/>
       </geometry>
     </collision>
@@ -80,5 +99,5 @@
   </link>
   <joint type="revolute" name="left_wheel_hinge">
-    <origin xyz="0 0.15 0.075" rpy="0 0 0"/>
+    <origin xyz="0.06 0.288 0.1518" rpy="0 0 0"/>
     <child link="left_wheel">left_wheel</child>
     <parent link="base_link">base_link</parent>
@@ -90,10 +109,10 @@
       <origin xyz="0 0.0 0" rpy="0 1.5707 1.5707"/>
       <geometry>
-        <cylinder  length="0.03" radius="0.0725"/>
+        <cylinder  length="0.03" radius="0.151"/>
       </geometry>
     </visual>
   </link>
   <joint type="fixed" name="visual_right_wheel_hinge">
-    <origin xyz="0.15 -0.15 0.075" rpy="0 0 0"/>
+    <origin xyz="0.06 -0.288 0.1518" rpy="0 0 0"/>
     <child link="visual_right_wheel">visual_right_wheel</child>
     <parent link="base_link">base_link</parent>
@@ -104,5 +123,5 @@
       <origin xyz="0 0.0 0" rpy="0 1.5707 1.5707"/>
       <geometry>
-         <cylinder  length="0.03" radius="0.0725"/>
+         <cylinder  length="0.03" radius="0.151"/>
       </geometry>
     </collision>
@@ -120,5 +139,5 @@
   </link>
   <joint type="revolute" name="right_wheel_hinge">
-    <origin xyz="0 -0.15 0.075" rpy="0 0 0"/>
+    <origin xyz="0.06 -0.288 0.1518" rpy="0 0 0"/>
     <child link="right_wheel">right_wheel</child>
     <parent link="base_link">base_link</parent>

File: orne_description/urdf/orne_middle.xacro (robot description, xacro)
@@ -8,5 +8,5 @@
 <xacro:include filename="$(find icart_mini_description)/urdf/sensors/hokuyo.urdf.xacro"/>
 <xacro:sensor_hokuyo name="hokuyo" parent="base_link">
-    <origin xyz="0.243 0 0.2" rpy="0 0 0"/>
+    <origin xyz="0.20 0 0.220" rpy="0 0 0"/>
 </xacro:sensor_hokuyo>
 </robot>

Commit message: Fix icart-middle.xacro wheel tread lenght

File: orne_description/urdf/icart_middle.xacro (robot description, xacro)
@@ -74,5 +74,5 @@
   </link>
   <joint type="fixed" name="visual_left_wheel_hinge">
-    <origin xyz="0.06 0.288 0.1518" rpy="0 0 0"/>
+    <origin xyz="0.06 0.22479 0.1518" rpy="0 0 0"/>
     <child link="visual_left_wheel">visual_left_wheel</child>
     <parent link="base_link">base_link</parent>
@@ -99,5 +99,5 @@
   </link>
   <joint type="revolute" name="left_wheel_hinge">
-    <origin xyz="0.06 0.288 0.1518" rpy="0 0 0"/>
+    <origin xyz="0.06 0.22479 0.1518" rpy="0 0 0"/>
     <child link="left_wheel">left_wheel</child>
     <parent link="base_link">base_link</parent>
@@ -114,5 +114,5 @@
   </link>
   <joint type="fixed" name="visual_right_wheel_hinge">
-    <origin xyz="0.06 -0.288 0.1518" rpy="0 0 0"/>
+    <origin xyz="0.06 -0.22479 0.1518" rpy="0 0 0"/>
     <child link="visual_right_wheel">visual_right_wheel</child>
     <parent link="base_link">base_link</parent>
@@ -139,5 +139,5 @@
   </link>
   <joint type="revolute" name="right_wheel_hinge">
-    <origin xyz="0.06 -0.288 0.1518" rpy="0 0 0"/>
+    <origin xyz="0.06 -0.22479 0.1518" rpy="0 0 0"/>
     <child link="right_wheel">right_wheel</child>
     <parent link="base_link">base_link</parent>

Commit message: change tread

File: orne_description/urdf/icart_middle.xacro (robot description, xacro)
@@ -74,5 +74,5 @@
   </link>
   <joint type="fixed" name="visual_left_wheel_hinge">
-    <origin xyz="0.06 0.22479 0.1518" rpy="0 0 0"/>
+    <origin xyz="0.06 0.199796 0.1518" rpy="0 0 0"/>
     <child link="visual_left_wheel">visual_left_wheel</child>
     <parent link="base_link">base_link</parent>
@@ -99,5 +99,5 @@
   </link>
   <joint type="revolute" name="left_wheel_hinge">
-    <origin xyz="0.06 0.22479 0.1518" rpy="0 0 0"/>
+    <origin xyz="0.06 0.199796 0.1518" rpy="0 0 0"/>
     <child link="left_wheel">left_wheel</child>
     <parent link="base_link">base_link</parent>
@@ -114,5 +114,5 @@
   </link>
   <joint type="fixed" name="visual_right_wheel_hinge">
-    <origin xyz="0.06 -0.22479 0.1518" rpy="0 0 0"/>
+    <origin xyz="0.06 -0.199796 0.1518" rpy="0 0 0"/>
     <child link="visual_right_wheel">visual_right_wheel</child>
     <parent link="base_link">base_link</parent>
@@ -139,5 +139,5 @@
   </link>
   <joint type="revolute" name="right_wheel_hinge">
-    <origin xyz="0.06 -0.22479 0.1518" rpy="0 0 0"/>
+    <origin xyz="0.06 -0.199796 0.1518" rpy="0 0 0"/>
     <child link="right_wheel">right_wheel</child>
     <parent link="base_link">base_link</parent>

Commit message: Change box size

File: orne_description/urdf/icart_middle.xacro (robot description, xacro)
@@ -12,5 +12,5 @@
       <origin xyz="0 0 0.1" rpy="0 0 0"/>
       <geometry>
-	<box size=".462 .50 .134"/>
+	<box size=".462 .45 .134"/>
       </geometry>
     </collision>
@@ -18,5 +18,5 @@
       <origin xyz="0 0 0.1" rpy="0 0 0"/>
       <geometry>
-	<box size=".462 .50 .134"/>
+	<box size=".462 .45 .134"/>
       </geometry>
       <material name="orange"/>
@@ -25,5 +25,5 @@
       <origin xyz="-0.095 0 0.305" rpy="0 0 0"/>
       <geometry>
-	<box size=".276 .50 .342"/>
+	<box size=".276 .45 .342"/>
       </geometry>
     </collision>
@@ -31,5 +31,5 @@
       <origin xyz="-0.095 0 0.305" rpy="0 0 0"/>
       <geometry>
-	<box size=".276 .50 .342"/>
+	<box size=".276 .45 .342"/>
       </geometry>
       <material name="orange"/>

Commit message: Gazeboで挙動がおかしかったので適当にInertiaをいじった

File: orne_description/urdf/icart_middle.xacro (robot description, xacro)
@@ -60,5 +60,5 @@
     </visual>
     <inertial>
-       <mass value="20" />
+       <mass value="15" />
        <origin xyz="0 0 0" rpy="0 0 0"/>
        <inertia ixx="1" ixy="0" ixz="0" iyy="1" iyz="0" izz="1" />
