Commit message: fix the imu position following a real robot

File: orne_description/urdf/orne_alpha.xacro (robot description, xacro)
@@ -4,6 +4,6 @@
 <xacro:include filename="$(find icart_mini_description)/urdf/icart_mini.gazebo"/>
 <xacro:include filename="$(find icart_mini_description)/urdf/sensors/imu.urdf.xacro"/>
-<xacro:sensor_imu name="imu" parent="base_link" size="0.1 0.1 0.1">
-    <origin xyz="-0.18 0.0 0.170" rpy="0 0 0"/>
+<xacro:sensor_imu name="imu" parent="base_link" size="0.05 0.05 0.05">
+    <origin xyz="0.19 0.0 0.15" rpy="0 0 0"/>
 </xacro:sensor_imu>
 <xacro:include filename="$(find icart_mini_description)/urdf/sensors/hokuyo3d.urdf.xacro"/>

Commit message: part sensor_hokuyo frame

File: orne_description/urdf/orne_alpha.xacro (robot description, xacro)
@@ -6,4 +6,8 @@
     <origin xyz="0.19 0.0 0.15" rpy="0 0 0"/>
 </xacro:sensor_imu>
+<xacro:include filename="$(find icart_mini_description)/urdf/sensors/hokuyo.urdf.xacro"/>
+<xacro:sensor_hokuyo name="hokuyo" parent="base_link">
+    <origin xyz="0.243 0 0.2" rpy="0 0 0"/>
+</xacro:sensor_hokuyo>
 <xacro:include filename="$(find icart_mini_description)/urdf/sensors/hokuyo3d.urdf.xacro"/>
 <xacro:sensor_hokuyo3d name="hokuyo3d" parent="base_link">

File: orne_description/urdf/orne_beta.xacro (robot description, xacro)
@@ -6,3 +6,7 @@
     <origin xyz="0.19 0.0 0.15" rpy="0 0 0"/>
 </xacro:sensor_imu>
+<xacro:include filename="$(find icart_mini_description)/urdf/sensors/hokuyo.urdf.xacro"/>
+<xacro:sensor_hokuyo name="hokuyo" parent="base_link">
+    <origin xyz="0.243 0 0.2" rpy="0 0 0"/>
+</xacro:sensor_hokuyo>
 </robot>

Commit message: respond to changes icart_mini.xacor for orne_alpha

File: orne_description/urdf/orne_alpha.xacro (robot description, xacro)
@@ -4,13 +4,13 @@
 <xacro:include filename="$(find icart_mini_description)/urdf/sensors/imu.urdf.xacro"/>
 <xacro:sensor_imu name="imu" parent="base_link" size="0.05 0.05 0.05">
-    <origin xyz="0.19 0.0 0.15" rpy="0 0 0"/>
+    <origin xyz="0.04 0.0 0.15" rpy="0 0 0"/>
 </xacro:sensor_imu>
 <xacro:include filename="$(find icart_mini_description)/urdf/sensors/hokuyo.urdf.xacro"/>
 <xacro:sensor_hokuyo name="hokuyo" parent="base_link">
-    <origin xyz="0.243 0 0.2" rpy="0 0 0"/>
+    <origin xyz="0.093 0 0.2" rpy="0 0 0"/>
 </xacro:sensor_hokuyo>
 <xacro:include filename="$(find icart_mini_description)/urdf/sensors/hokuyo3d.urdf.xacro"/>
 <xacro:sensor_hokuyo3d name="hokuyo3d" parent="base_link">
-    <origin xyz="0.27 0 0.35" rpy="0 0.192 0"/>
+    <origin xyz="0.12 0 0.35" rpy="0 0.192 0"/>
 </xacro:sensor_hokuyo3d>
 </robot>

Commit message: Revert "merge indigo-devel"
This reverts commit bb399b80f1d239dc8bbc194c85311abb39243b29, reversing
changes made to be4770382bcc0c9787cba605e7f6124608b2d76e.

File: orne_description/urdf/orne_alpha.xacro (robot description, xacro)
@@ -4,13 +4,13 @@
 <xacro:include filename="$(find icart_mini_description)/urdf/sensors/imu.urdf.xacro"/>
 <xacro:sensor_imu name="imu" parent="base_link" size="0.05 0.05 0.05">
-    <origin xyz="0.04 0.0 0.15" rpy="0 0 0"/>
+    <origin xyz="0.19 0.0 0.15" rpy="0 0 0"/>
 </xacro:sensor_imu>
 <xacro:include filename="$(find icart_mini_description)/urdf/sensors/hokuyo.urdf.xacro"/>
 <xacro:sensor_hokuyo name="hokuyo" parent="base_link">
-    <origin xyz="0.093 0 0.2" rpy="0 0 0"/>
+    <origin xyz="0.243 0 0.2" rpy="0 0 0"/>
 </xacro:sensor_hokuyo>
 <xacro:include filename="$(find icart_mini_description)/urdf/sensors/hokuyo3d.urdf.xacro"/>
 <xacro:sensor_hokuyo3d name="hokuyo3d" parent="base_link">
-    <origin xyz="0.12 0 0.35" rpy="0 0.192 0"/>
+    <origin xyz="0.27 0 0.35" rpy="0 0.192 0"/>
 </xacro:sensor_hokuyo3d>
 </robot>

File: orne_description/urdf/orne_beta.xacro (robot description, xacro)
@@ -4,13 +4,9 @@
 <xacro:include filename="$(find icart_mini_description)/urdf/sensors/imu.urdf.xacro"/>
 <xacro:sensor_imu name="imu" parent="base_link" size="0.05 0.05 0.05">
-    <origin xyz="0.04 0.0 0.15" rpy="0 0 0"/>
+    <origin xyz="0.19 0.0 0.15" rpy="0 0 0"/>
 </xacro:sensor_imu>
 <xacro:include filename="$(find icart_mini_description)/urdf/sensors/hokuyo.urdf.xacro"/>
 <xacro:sensor_hokuyo name="hokuyo" parent="base_link">
-<<<<<<< HEAD
     <origin xyz="0.20 0 0.220" rpy="0 0 0"/>
-=======
-    <origin xyz="0.093 0 0.2" rpy="0 0 0"/>
->>>>>>> indigo-devel
 </xacro:sensor_hokuyo>
 </robot>

Commit message: fix xacro

File: orne_description/urdf/orne_alpha.xacro (robot description, xacro)
@@ -4,13 +4,13 @@
 <xacro:include filename="$(find icart_mini_description)/urdf/sensors/imu.urdf.xacro"/>
 <xacro:sensor_imu name="imu" parent="base_link" size="0.05 0.05 0.05">
-    <origin xyz="0.19 0.0 0.15" rpy="0 0 0"/>
+    <origin xyz="0.04 0.0 0.15" rpy="0 0 0"/>
 </xacro:sensor_imu>
 <xacro:include filename="$(find icart_mini_description)/urdf/sensors/hokuyo.urdf.xacro"/>
 <xacro:sensor_hokuyo name="hokuyo" parent="base_link">
-    <origin xyz="0.243 0 0.2" rpy="0 0 0"/>
+    <origin xyz="0.93 0 0.2" rpy="0 0 0"/>
 </xacro:sensor_hokuyo>
 <xacro:include filename="$(find icart_mini_description)/urdf/sensors/hokuyo3d.urdf.xacro"/>
 <xacro:sensor_hokuyo3d name="hokuyo3d" parent="base_link">
-    <origin xyz="0.27 0 0.35" rpy="0 0.192 0"/>
+    <origin xyz="0.12 0 0.35" rpy="0 0.192 0"/>
 </xacro:sensor_hokuyo3d>
 </robot>

File: orne_description/urdf/orne_beta.xacro (robot description, xacro)
@@ -4,9 +4,9 @@
 <xacro:include filename="$(find icart_mini_description)/urdf/sensors/imu.urdf.xacro"/>
 <xacro:sensor_imu name="imu" parent="base_link" size="0.05 0.05 0.05">
-    <origin xyz="0.19 0.0 0.15" rpy="0 0 0"/>
+    <origin xyz="0.04 0.0 0.15" rpy="0 0 0"/>
 </xacro:sensor_imu>
 <xacro:include filename="$(find icart_mini_description)/urdf/sensors/hokuyo.urdf.xacro"/>
 <xacro:sensor_hokuyo name="hokuyo" parent="base_link">
-    <origin xyz="0.20 0 0.220" rpy="0 0 0"/>
+    <origin xyz="0.2 0 0.2" rpy="0 0 0"/>
 </xacro:sensor_hokuyo>
 </robot>

Commit message: urgの位置を修正

File: orne_description/urdf/orne_alpha.xacro (robot description, xacro)
@@ -8,5 +8,5 @@
 <xacro:include filename="$(find icart_mini_description)/urdf/sensors/hokuyo.urdf.xacro"/>
 <xacro:sensor_hokuyo name="hokuyo" parent="base_link">
-    <origin xyz="0.93 0 0.2" rpy="0 0 0"/>
+    <origin xyz="0.093 0 0.2" rpy="0 0 0"/>
 </xacro:sensor_hokuyo>
 <xacro:include filename="$(find icart_mini_description)/urdf/sensors/hokuyo3d.urdf.xacro"/>

Commit message: add diagonally fixed 2DURG parameter to orne_alpha.xacro,launch

File: orne_description/urdf/orne_alpha.xacro (robot description, xacro)
@@ -10,4 +10,8 @@
     <origin xyz="0.093 0 0.2" rpy="0 0 0"/>
 </xacro:sensor_hokuyo>
+<xacro:include filename="$(find icart_mini_description)/urdf/sensors/hokuyo.urdf.xacro"/>
+<xacro:sensor_hokuyo name="diagonally_hokuyo" parent="base_link">
+   <origin xyz="0.093 0 0.4" rpy="0 0.296706 0"/> <!-- 0.296706 radian = 17 degree -->
+</xacro:sensor_hokuyo>
 <xacro:include filename="$(find icart_mini_description)/urdf/sensors/hokuyo3d.urdf.xacro"/>
 <xacro:sensor_hokuyo3d name="hokuyo3d" parent="base_link">

Commit message: modify orne_description/urdf/orne_alpha.xacro

File: orne_description/urdf/orne_alpha.xacro (robot description, xacro)
@@ -2,15 +2,18 @@
 <robot name="orne_alpha" xmlns:xacro="http://www.ros.org/wiki/xacro">
 <xacro:include filename="$(find icart_mini_description)/urdf/icart_mini.xacro"/>
+<!-- Setting for imu -->
 <xacro:include filename="$(find icart_mini_description)/urdf/sensors/imu.urdf.xacro"/>
 <xacro:sensor_imu name="imu" parent="base_link" size="0.05 0.05 0.05">
     <origin xyz="0.04 0.0 0.15" rpy="0 0 0"/>
 </xacro:sensor_imu>
+<!-- Setting for levelly fixed 2D URG -->
 <xacro:include filename="$(find icart_mini_description)/urdf/sensors/hokuyo.urdf.xacro"/>
 <xacro:sensor_hokuyo name="hokuyo" parent="base_link">
     <origin xyz="0.093 0 0.2" rpy="0 0 0"/>
 </xacro:sensor_hokuyo>
+<!-- Setting for diagonally fixed 2D URG -->
 <xacro:include filename="$(find icart_mini_description)/urdf/sensors/hokuyo.urdf.xacro"/>
 <xacro:sensor_hokuyo name="diagonally_hokuyo" parent="base_link">
-   <origin xyz="0.093 0 0.4" rpy="0 0.296706 0"/> <!-- 0.296706 radian = 17 degree -->
+   <origin xyz="0.093 0 0.427" rpy="0 0.296706 0"/> <!-- 0.296706 radian = 17 degree -->
 </xacro:sensor_hokuyo>
 <!--

Commit message: modify orne_alpha.launch and orne_alpha.xacro

File: orne_description/urdf/orne_alpha.xacro (robot description, xacro)
@@ -15,5 +15,5 @@
 <xacro:include filename="$(find icart_mini_description)/urdf/sensors/hokuyo.urdf.xacro"/>
 <xacro:sensor_hokuyo name="diagonally_hokuyo" parent="base_link">
-   <origin xyz="0.093 0 0.427" rpy="0 0.296706 0"/> <!-- 0.296706 radian = 17 degree -->
+   <origin xyz="0.093 0 0.664" rpy="0 0.296706 0"/> <!-- 0.296706 radian = 17 degree -->
 </xacro:sensor_hokuyo>
 <!--

Commit message: x用のパラメータファイルの追加

File: orne_description/urdf/orne_alpha.xacro (robot description, xacro)
@@ -1,19 +1,19 @@
 <?xml version="1.0"?>
 <robot name="orne_alpha" xmlns:xacro="http://www.ros.org/wiki/xacro">
-<xacro:include filename="$(find icart_mini_description)/urdf/icart_mini.xacro"/>
+  <xacro:include filename="$(find orne_description)/urdf/orne_x.xacro"/>
 <!-- Setting for imu -->
 <xacro:include filename="$(find icart_mini_description)/urdf/sensors/imu.urdf.xacro"/>
 <xacro:sensor_imu name="imu" parent="base_link" size="0.05 0.05 0.05">
-    <origin xyz="0.04 0.0 0.15" rpy="0 0 0"/>
+    <origin xyz="-0.145 0.0 0.15" rpy="0 0 0"/>
 </xacro:sensor_imu>
 <!-- Setting for levelly fixed 2D URG -->
 <xacro:include filename="$(find icart_mini_description)/urdf/sensors/hokuyo.urdf.xacro"/>
 <xacro:sensor_hokuyo name="hokuyo" parent="base_link">
-    <origin xyz="0.093 0 0.2" rpy="0 0 0"/>
+    <origin xyz="0.212 0 0.0985" rpy="0 0 0"/>
 </xacro:sensor_hokuyo>
 <!-- Setting for diagonally fixed 2D URG -->
 <xacro:include filename="$(find icart_mini_description)/urdf/sensors/hokuyo.urdf.xacro"/>
 <xacro:sensor_hokuyo name="diagonally_hokuyo" parent="base_link">
-   <origin xyz="0.093 0 0.664" rpy="0 0.296706 0"/> <!-- 0.296706 radian = 17 degree -->
+   <origin xyz="0.098 0 0.422" rpy="0 0.296706 0"/> <!-- 0.296706 radian = 17 degree -->
 </xacro:sensor_hokuyo>
 <!--

Commit message: change description

File: orne_description/urdf/orne_alpha.xacro (robot description, xacro)
@@ -5,10 +5,10 @@
 <xacro:include filename="$(find icart_mini_description)/urdf/sensors/imu.urdf.xacro"/>
 <xacro:sensor_imu name="imu" parent="base_link" size="0.05 0.05 0.05">
-    <origin xyz="-0.145 0.0 0.15" rpy="0 0 0"/>
+    <origin xyz="-0.145 0.0 0.21" rpy="0 0 0"/>
 </xacro:sensor_imu>
 <!-- Setting for levelly fixed 2D URG -->
 <xacro:include filename="$(find icart_mini_description)/urdf/sensors/hokuyo.urdf.xacro"/>
 <xacro:sensor_hokuyo name="hokuyo" parent="base_link">
-    <origin xyz="0.212 0 0.0985" rpy="0 0 0"/>
+    <origin xyz="0.212 0 0.2485" rpy="0 0 0"/>
 </xacro:sensor_hokuyo>
 <!-- Setting for diagonally fixed 2D URG -->

File: orne_description/urdf/orne_x.xacro (robot description, xacro)
@@ -12,5 +12,5 @@
       <origin xyz="0 0 0.1" rpy="0 0 0"/>
       <geometry>
-	<box size=".462 .45 .134"/>
+	<box size=".40 .45 .134"/>
       </geometry>
     </collision>
@@ -25,5 +25,5 @@
       <origin xyz="-0.095 0 0.305" rpy="0 0 0"/>
       <geometry>
-	<box size=".276 .45 .342"/>
+	<box size=".376 .45 .242"/>
       </geometry>
     </collision>
@@ -36,25 +36,25 @@
     </visual>
     <collision name="collision">
-      <origin xyz="-0.231 -0.141 0.05" rpy="0 1.5707 1.5707"/>
+      <origin xyz="0.201 -0.141 0.075" rpy="0 1.5707 1.5707"/>
       <geometry>
-        <cylinder  length="0.03" radius="0.04625"/>
+        <cylinder  length="0.03" radius="0.075"/>
       </geometry>
     </collision>
     <visual name="visual">
-      <origin xyz="-0.231 -0.141 0.05" rpy="0 1.5707 1.5707"/>
+      <origin xyz="0.201 -0.141 0.075" rpy="0 1.5707 1.5707"/>
       <geometry>
-        <cylinder  length="0.03" radius="0.04625"/>
+        <cylinder  length="0.03" radius="0.075"/>
       </geometry>
     </visual>
     <collision name="collision">
-      <origin xyz="-0.231 0.141 0.05" rpy="0 1.5707 1.5707"/>
+      <origin xyz="0.201 0.141 0.075" rpy="0 1.5707 1.5707"/>
       <geometry>
-        <cylinder  length="0.03" radius="0.04625"/>
+        <cylinder  length="0.03" radius="0.075"/>
       </geometry>
     </collision>
     <visual name="visual">
-      <origin xyz="-0.231 0.141 0.05" rpy="0 1.5707 1.5707"/>
+      <origin xyz="0.201 0.141 0.075" rpy="0 1.5707 1.5707"/>
       <geometry>
-        <cylinder  length="0.03" radius="0.04625"/>
+        <cylinder  length="0.03" radius="0.075"/>
       </geometry>
     </visual>
@@ -62,5 +62,5 @@
        <mass value="15" />
        <origin xyz="0 0 0" rpy="0 0 0"/>
-       <inertia ixx="1" ixy="0" ixz="0" iyy="1" iyz="0" izz="1" />
+       <inertia ixx="0.1" ixy="0" ixz="0" iyy="0.1" iyz="0" izz="0.1" />
     </inertial>
   </link>
@@ -74,5 +74,5 @@
   </link>
   <joint type="fixed" name="visual_left_wheel_hinge">
-    <origin xyz="-0.145 0.223 0.15" rpy="0 0 0"/>
+    <origin xyz="-0.145 0.233 0.15" rpy="0 0 0"/>
     <child link="visual_left_wheel">visual_left_wheel</child>
     <parent link="base_link">base_link</parent>
@@ -89,5 +89,5 @@
       <origin xyz="0 0.0 0" rpy="0 1.5707 1.5707"/>
       <geometry>
-        <cylinder  length="0.03" radius="0.0725"/>
+        <cylinder  length="0.03" radius="0.151"/>
       </geometry>
     </visual-->
@@ -99,5 +99,5 @@
   </link>
   <joint type="revolute" name="left_wheel_hinge">
-    <origin xyz="-0.145 0.2228 0.15" rpy="0 0 0"/>
+    <origin xyz="-0.145 0.223 0.15" rpy="0 0 0"/>
     <child link="left_wheel">left_wheel</child>
     <parent link="base_link">base_link</parent>
@@ -114,5 +114,5 @@
   </link>
   <joint type="fixed" name="visual_right_wheel_hinge">
-    <origin xyz="-0.145 -0.2228 0.15" rpy="0 0 0"/>
+    <origin xyz="-0.145 -0.223 0.15" rpy="0 0 0"/>
     <child link="visual_right_wheel">visual_right_wheel</child>
     <parent link="base_link">base_link</parent>
@@ -129,5 +129,5 @@
       <origin xyz="0 0.0 0" rpy="0 1.5707 1.5707"/>
       <geometry>
-        <cylinder  length="0.03" radius="0.0725"/>
+        <cylinder  length="0.03" radius="0.151"/>
       </geometry>
     </visual-->
@@ -139,5 +139,5 @@
   </link>
   <joint type="revolute" name="right_wheel_hinge">
-    <origin xyz="-0.145 -0.2228 0.15" rpy="0 0 0"/>
+    <origin xyz="-0.145 -0.223 0.15" rpy="0 0 0"/>
     <child link="right_wheel">right_wheel</child>
     <parent link="base_link">base_link</parent>

Commit message: inertialの変更

File: orne_description/urdf/orne_alpha.xacro (robot description, xacro)
@@ -5,15 +5,15 @@
 <xacro:include filename="$(find icart_mini_description)/urdf/sensors/imu.urdf.xacro"/>
 <xacro:sensor_imu name="imu" parent="base_link" size="0.05 0.05 0.05">
-    <origin xyz="-0.145 0.0 0.21" rpy="0 0 0"/>
+    <origin xyz="-0.145 0.0 0.15" rpy="0 0 0"/>
 </xacro:sensor_imu>
 <!-- Setting for levelly fixed 2D URG -->
 <xacro:include filename="$(find icart_mini_description)/urdf/sensors/hokuyo.urdf.xacro"/>
 <xacro:sensor_hokuyo name="hokuyo" parent="base_link">
-    <origin xyz="0.212 0 0.2485" rpy="0 0 0"/>
+    <origin xyz="0.212 0 0.235" rpy="0 0 0"/>
 </xacro:sensor_hokuyo>
 <!-- Setting for diagonally fixed 2D URG -->
 <xacro:include filename="$(find icart_mini_description)/urdf/sensors/hokuyo.urdf.xacro"/>
 <xacro:sensor_hokuyo name="diagonally_hokuyo" parent="base_link">
-   <origin xyz="0.098 0 0.422" rpy="0 0.296706 0"/> <!-- 0.296706 radian = 17 degree -->
+   <origin xyz="0.098 0 0.447" rpy="0 0.296706 0"/> <!-- 0.296706 radian = 17 degree -->
 </xacro:sensor_hokuyo>
 <!--

File: orne_description/urdf/orne_x.xacro (robot description, xacro)
@@ -12,5 +12,5 @@
       <origin xyz="0 0 0.1" rpy="0 0 0"/>
       <geometry>
-	<box size=".40 .45 .134"/>
+	<box size=".462 .40 .134"/>
       </geometry>
     </collision>
@@ -18,43 +18,43 @@
       <origin xyz="0 0 0.1" rpy="0 0 0"/>
       <geometry>
-	<box size=".462 .45 .134"/>
+	<box size=".462 .40 .134"/>
       </geometry>
       <material name="orange"/>
     </visual>
     <collision>
-      <origin xyz="-0.095 0 0.305" rpy="0 0 0"/>
+      <origin xyz="-0.095 0 0.245" rpy="0 0 0"/>
       <geometry>
-	<box size=".376 .45 .242"/>
+	<box size=".25 .40 .255"/>
       </geometry>
     </collision>
     <visual>
-      <origin xyz="-0.095 0 0.305" rpy="0 0 0"/>
+      <origin xyz="-0.095 0 0.285" rpy="0 0 0"/>
       <geometry>
-	<box size=".276 .45 .342"/>
+	<box size=".25 .40 .255"/>
       </geometry>
       <material name="orange"/>
     </visual>
     <collision name="collision">
-      <origin xyz="0.201 -0.141 0.075" rpy="0 1.5707 1.5707"/>
+      <origin xyz="0.201 -0.141 0.05" rpy="0 1.5707 1.5707"/>
       <geometry>
-        <cylinder  length="0.03" radius="0.075"/>
+        <cylinder  length="0.03" radius="0.04625"/>
       </geometry>
     </collision>
     <visual name="visual">
-      <origin xyz="0.201 -0.141 0.075" rpy="0 1.5707 1.5707"/>
+      <origin xyz="0.201 -0.141 0.05" rpy="0 1.5707 1.5707"/>
       <geometry>
-        <cylinder  length="0.03" radius="0.075"/>
+        <cylinder  length="0.03" radius="0.04625"/>
       </geometry>
     </visual>
     <collision name="collision">
-      <origin xyz="0.201 0.141 0.075" rpy="0 1.5707 1.5707"/>
+      <origin xyz="0.201 0.141 0.05" rpy="0 1.5707 1.5707"/>
       <geometry>
-        <cylinder  length="0.03" radius="0.075"/>
+        <cylinder  length="0.03" radius="0.04625"/>
       </geometry>
     </collision>
     <visual name="visual">
-      <origin xyz="0.201 0.141 0.075" rpy="0 1.5707 1.5707"/>
+      <origin xyz="0.201 0.141 0.05" rpy="0 1.5707 1.5707"/>
       <geometry>
-        <cylinder  length="0.03" radius="0.075"/>
+        <cylinder  length="0.03" radius="0.04625"/>
       </geometry>
     </visual>
@@ -62,5 +62,5 @@
        <mass value="15" />
        <origin xyz="0 0 0" rpy="0 0 0"/>
-       <inertia ixx="0.1" ixy="0" ixz="0" iyy="0.1" iyz="0" izz="0.1" />
+       <inertia ixx="1" ixy="0" ixz="0" iyy="1" iyz="0" izz="1" />
     </inertial>
   </link>
@@ -74,5 +74,5 @@
   </link>
   <joint type="fixed" name="visual_left_wheel_hinge">
-    <origin xyz="-0.145 0.233 0.15" rpy="0 0 0"/>
+    <origin xyz="-0.145 0.223 0.1518" rpy="0 0 0"/>
     <child link="visual_left_wheel">visual_left_wheel</child>
     <parent link="base_link">base_link</parent>
@@ -81,5 +81,5 @@
   <link name="left_wheel">
     <collision name="collision">
-      <origin xyz="0 0.0 0" rpy="0 0 0"/>
+      <origin xyz="0 0.0 0" rpy="0 1.5707 1.5707"/>
       <geometry>
          <cylinder  length="0.03" radius="0.151"/>
@@ -89,9 +89,9 @@
       <origin xyz="0 0.0 0" rpy="0 1.5707 1.5707"/>
       <geometry>
-        <cylinder  length="0.03" radius="0.151"/>
+        <cylinder  length="0.03" radius="0.0725"/>
       </geometry>
     </visual-->
     <inertial>
-      <mass value="1" />
+      <mass value="5" />
       <origin xyz="0 0.0 0"/>
       <inertia ixx="0.1" ixy="0" ixz="0" iyy="0.1" iyz="0" izz="0.1" />
@@ -99,5 +99,5 @@
   </link>
   <joint type="revolute" name="left_wheel_hinge">
-    <origin xyz="-0.145 0.223 0.15" rpy="0 0 0"/>
+    <origin xyz="-0.145 0.2228 0.1518" rpy="0 0 0"/>
     <child link="left_wheel">left_wheel</child>
     <parent link="base_link">base_link</parent>
@@ -114,5 +114,5 @@
   </link>
   <joint type="fixed" name="visual_right_wheel_hinge">
-    <origin xyz="-0.145 -0.223 0.15" rpy="0 0 0"/>
+    <origin xyz="-0.145 -0.2228 0.1518" rpy="0 0 0"/>
     <child link="visual_right_wheel">visual_right_wheel</child>
     <parent link="base_link">base_link</parent>
@@ -129,9 +129,9 @@
       <origin xyz="0 0.0 0" rpy="0 1.5707 1.5707"/>
       <geometry>
-        <cylinder  length="0.03" radius="0.151"/>
+        <cylinder  length="0.03" radius="0.0725"/>
       </geometry>
     </visual-->
     <inertial>
-      <mass value="1" />
+      <mass value="5" />
       <origin xyz="0 0.0 0"/>
       <inertia ixx="0.1" ixy="0" ixz="0" iyy="0.1" iyz="0" izz="0.1" />
@@ -139,5 +139,5 @@
   </link>
   <joint type="revolute" name="right_wheel_hinge">
-    <origin xyz="-0.145 -0.223 0.15" rpy="0 0 0"/>
+    <origin xyz="-0.145 -0.2228 0.1518" rpy="0 0 0"/>
     <child link="right_wheel">right_wheel</child>
     <parent link="base_link">base_link</parent>

Commit message: working

File: orne_description/urdf/orne_alpha.xacro (robot description, xacro)
@@ -1,5 +1,5 @@
 <?xml version="1.0"?>
 <robot name="orne_alpha" xmlns:xacro="http://www.ros.org/wiki/xacro">
-  <xacro:include filename="$(find orne_description)/urdf/orne_x.xacro"/>
+<xacro:include filename="$(find orne_description)/urdf/orne_x.xacro"/>
 <!-- Setting for imu -->
 <xacro:include filename="$(find icart_mini_description)/urdf/sensors/imu.urdf.xacro"/>

File: orne_description/urdf/orne_x.xacro (robot description, xacro)
@@ -1,10 +1,10 @@
 <?xml version="1.0"?>
 <!-- Revolute-Revolute Manipulator -->
-<robot name="icart_middle" xmlns:xacro="http://www.ros.org/wiki/xacro">
+<robot name="orne_x" xmlns:xacro="http://www.ros.org/wiki/xacro">
   <!-- Constants for robot dimensions -->
   <xacro:property name="PI" value="3.1415926535897931"/>
   <!-- Import Rviz colors -->
   <xacro:include filename="$(find icart_mini_description)/urdf/materials.xacro" />
-  <xacro:include filename="$(find orne_description)/urdf/icart_middle.gazebo"/>
+  <xacro:include filename="$(find orne_description)/urdf/orne_x.gazebo"/>
   <!-- Base Link -->
   <link name="base_link">
@@ -18,5 +18,5 @@
       <origin xyz="0 0 0.1" rpy="0 0 0"/>
       <geometry>
-	<box size=".462 .45 .134"/>
+	<box size=".40 .45 .134"/>
       </geometry>
       <material name="orange"/>
@@ -31,5 +31,5 @@
       <origin xyz="-0.095 0 0.305" rpy="0 0 0"/>
       <geometry>
-	<box size=".276 .45 .342"/>
+	<box size=".376 .45 .242"/>
       </geometry>
       <material name="orange"/>
@@ -62,5 +62,5 @@
        <mass value="15" />
        <origin xyz="0 0 0" rpy="0 0 0"/>
-       <inertia ixx="0.1" ixy="0" ixz="0" iyy="0.1" iyz="0" izz="0.1" />
+       <inertia ixx="1" ixy="0" ixz="0" iyy="1" iyz="0" izz="1" />
     </inertial>
   </link>
@@ -81,5 +81,5 @@
   <link name="left_wheel">
     <collision name="collision">
-      <origin xyz="0 0.0 0" rpy="0 0 0"/>
+      <origin xyz="0 0.0 0" rpy="0 1.5707 1.5707"/>
       <geometry>
          <cylinder  length="0.03" radius="0.151"/>
@@ -135,5 +135,5 @@
       <mass value="1" />
       <origin xyz="0 0.0 0"/>
-      <inertia ixx="0.1" ixy="0" ixz="0" iyy="0.1" iyz="0" izz="0.1" />
+      <inertia ixx="0.1" ixy="0" ixz="0" iyy="0.1" iyz="0" izz="1" />
     </inertial>
   </link>
