Commit message: change xacro namespace

File: orne_description/urdf/orne_alpha.xacro (robot description, xacro)
@@ -1,20 +1,24 @@
 <?xml version="1.0"?>
-<robot name="orne_alpha" xmlns:xacro="http://www.ros.org/wiki/xacro">
+<robot name="orne_alpha" xmlns:xacro="http://ros.org/wiki/xacro"
+                         xmlns:sensor="http://playerstage.sourceforge.net/gazebo/xmlschema/#sensor"
+                         xmlns:controller="http://playerstage.sourceforge.net/gazebo/xmlschema/#controller"
+                         xmlns:interface="http://playerstage.sourceforge.net/gazebo/xmlschema/#interface"
+>
 <xacro:include filename="$(find orne_description)/urdf/orne_x.xacro"/>
+<xacro:include filename="$(find icart_mini_description)/urdf/sensors/imu.urdf.xacro"/>
+<xacro:include filename="$(find icart_mini_description)/urdf/sensors/hokuyo.urdf.xacro"/>
 <!-- Setting for imu -->
-<xacro:include filename="$(find icart_mini_description)/urdf/sensors/imu.urdf.xacro"/>
 <xacro:sensor_imu name="imu" parent="base_link" size="0.05 0.05 0.05">
     <origin xyz="-0.145 0.0 0.21" rpy="0 0 0"/>
 </xacro:sensor_imu>
 <!-- Setting for levelly fixed 2D URG -->
-<xacro:include filename="$(find icart_mini_description)/urdf/sensors/hokuyo.urdf.xacro"/>
 <xacro:sensor_hokuyo name="hokuyo" parent="base_link">
     <origin xyz="0.212 0 0.2485" rpy="0 0 0"/>
 </xacro:sensor_hokuyo>
 <!-- Setting for diagonally fixed 2D URG -->
-<xacro:include filename="$(find icart_mini_description)/urdf/sensors/hokuyo.urdf.xacro"/>
+<!--xacro:include filename="$(find icart_mini_description)/urdf/sensors/hokuyo.urdf.xacro"/>
 <xacro:sensor_hokuyo name="diagonally_hokuyo" parent="base_link">
-   <origin xyz="0.098 0 0.422" rpy="0 0.296706 0"/> <!-- 0.296706 radian = 17 degree -->
-</xacro:sensor_hokuyo>
+   <origin xyz="0.098 0 0.422" rpy="0 0.296706 0"/>
+</xacro:sensor_hokuyo-->
 <!--
 <xacro:include filename="$(find icart_mini_description)/urdf/sensors/hokuyo3d.urdf.xacro"/>

File: orne_description/urdf/orne_x.xacro (robot description, xacro)
@@ -1,5 +1,5 @@
 <?xml version="1.0"?>
 <!-- Revolute-Revolute Manipulator -->
-<robot name="orne_x" xmlns:xacro="http://www.ros.org/wiki/xacro">
+<robot name="orne_x" xmlns:xacro="http://ros.org/wiki/xacro">
   <!-- Constants for robot dimensions -->
   <xacro:property name="PI" value="3.1415926535897931"/>

Commit message: gazeboでも動くようになった

File: orne_description/urdf/orne_alpha.xacro (robot description, xacro)
@@ -8,4 +8,5 @@
 <xacro:include filename="$(find icart_mini_description)/urdf/sensors/imu.urdf.xacro"/>
 <xacro:include filename="$(find icart_mini_description)/urdf/sensors/hokuyo.urdf.xacro"/>
+<xacro:include filename="$(find velodyne_description)/urdf/VLP-16.urdf.xacro"/>
 <!-- Setting for imu -->
 <xacro:sensor_imu name="imu" parent="base_link" size="0.05 0.05 0.05">
@@ -24,6 +25,10 @@
 <xacro:include filename="$(find icart_mini_description)/urdf/sensors/hokuyo3d.urdf.xacro"/>
 <xacro:sensor_hokuyo3d name="hokuyo3d" parent="base_link">
-    <origin xyz="0.12 0 0.35" rpy="0 0.192 0"/>
+    <origin xyz="0.2 0 0.7" rpy="0 0.174 0"/>
 </xacro:sensor_hokuyo3d>
 -->
+<xacro:include filename="$(find velodyne_description)/urdf/VLP-16.urdf.xacro"/>
+<xacro:VLP-16 name="velodyne" parent="base_link">
+    <origin xyz="0.098 0.0 0.422" rpy="0 0 0"/>
+</xacro:VLP-16>
 </robot>

Commit message: IMU用にα のセンセの角度と起動launchファイルの変更

File: orne_description/urdf/orne_alpha.xacro (robot description, xacro)
@@ -11,5 +11,5 @@
 <!-- Setting for imu -->
 <xacro:sensor_imu name="imu" parent="base_link" size="0.05 0.05 0.05">
-    <origin xyz="-0.145 0.0 0.21" rpy="0 0 0"/>
+    <origin xyz="-0.145 0.0 0.21" rpy="0 3.14 0"/>
 </xacro:sensor_imu>
 <!-- Setting for levelly fixed 2D URG -->

File: orne_description/urdf/orne_x.xacro (robot description, xacro)
@@ -36,5 +36,5 @@
     </visual>
     <collision name="collision">
-      <origin xyz="0.301 -0.141 0.075" rpy="0 1.5707 1.5707"/>
+      <origin xyz="0.301 -0.141 0.075" rpy="1.57 0 0"/>
       <geometry>
         <cylinder  length="0.03" radius="0.075"/>
@@ -42,5 +42,5 @@
     </collision>
     <visual name="visual">
-      <origin xyz="0.301 -0.141 0.075" rpy="0 1.5707 1.5707"/>
+      <origin xyz="0.301 -0.141 0.075" rpy="1.57 0 0"/>
       <geometry>
         <cylinder  length="0.03" radius="0.075"/>
@@ -48,5 +48,5 @@
     </visual>
     <collision name="collision">
-      <origin xyz="0.301 0.141 0.075" rpy="0 1.5707 1.5707"/>
+      <origin xyz="0.301 0.141 0.075" rpy="1.57 0 0"/>
       <geometry>
         <cylinder  length="0.03" radius="0.075"/>
@@ -54,5 +54,5 @@
     </collision>
     <visual name="visual">
-      <origin xyz="0.301 0.141 0.075" rpy="0 1.5707 1.5707"/>
+      <origin xyz="0.301 0.141 0.075" rpy="1.57 0 0"/>
       <geometry>
         <cylinder  length="0.03" radius="0.075"/>
@@ -67,5 +67,5 @@
   <link name="visual_left_wheel">
     <visual name="visual">
-      <origin xyz="0 0.0 0" rpy="0 1.5707 1.5707"/>
+      <origin xyz="0 0.0 0" rpy="1.57 0 0"/>
       <geometry>
         <cylinder  length="0.03" radius="0.151"/>
@@ -81,5 +81,5 @@
   <link name="left_wheel">
     <collision name="collision">
-      <origin xyz="0 0.0 0" rpy="0 1.5707 1.5707"/>
+      <origin xyz="0 0.0 0" rpy="1.57 0 0"/>
       <geometry>
          <cylinder  length="0.03" radius="0.151"/>
@@ -87,5 +87,5 @@
     </collision>
     <!--visual name="visual">
-      <origin xyz="0 0.0 0" rpy="0 1.5707 1.5707"/>
+      <origin xyz="0 0.0 0" rpy="0 0 0"/>
       <geometry>
         <cylinder  length="0.03" radius="0.0725"/>
@@ -107,5 +107,5 @@
   <link name="visual_right_wheel">
     <visual name="visual">
-      <origin xyz="0 0.0 0" rpy="0 1.5707 1.5707"/>
+      <origin xyz="0 0.0 0" rpy="1.57 0 0"/>
       <geometry>
         <cylinder  length="0.03" radius="0.151"/>
@@ -121,5 +121,5 @@
   <link name="right_wheel">
     <collision name="collision">
-      <origin xyz="0 0.0 0" rpy="0 1.5707 1.5707"/>
+      <origin xyz="0 0.0 0" rpy="1.57 00 00"/>
       <geometry>
          <cylinder  length="0.03" radius="0.151"/>
@@ -127,5 +127,5 @@
     </collision>
     <!--visual name="visual">
-      <origin xyz="0 0.0 0" rpy="0 1.5707 1.5707"/>
+      <origin xyz="0 0.0 0" rpy="0 0 0"/>
       <geometry>
         <cylinder  length="0.03" radius="0.0725"/>

Commit message: vlp16の傾きを変更した

File: orne_description/urdf/orne_alpha.xacro (robot description, xacro)
@@ -32,5 +32,5 @@
 <xacro:include filename="$(find velodyne_description)/urdf/VLP-16.urdf.xacro"/>
 <xacro:VLP-16 name="velodyne" parent="base_link">
-    <origin xyz="0.098 0.0 0.422" rpy="0 0 0"/>
+    <origin xyz="0.098 0.0 0.422" rpy="0 0 -0.12"/>
 </xacro:VLP-16>
 </robot>

Commit message: velodyne周りを修正

File: orne_description/urdf/orne_alpha.xacro (robot description, xacro)
@@ -8,5 +8,4 @@
 <xacro:include filename="$(find icart_mini_description)/urdf/sensors/imu.urdf.xacro"/>
 <xacro:include filename="$(find icart_mini_description)/urdf/sensors/hokuyo.urdf.xacro"/>
-<xacro:include filename="$(find velodyne_description)/urdf/VLP-16.urdf.xacro"/>
 <!-- Setting for imu -->
 <xacro:sensor_imu name="imu" parent="base_link" size="0.05 0.05 0.05">
@@ -30,5 +29,6 @@
 </xacro:sensor_hokuyo3d>
 -->
-<xacro:include filename="$(find velodyne_description)/urdf/VLP-16.urdf.xacro"/>
+<!--$acro:include filename="$(find velodyne_description)/urdf/VLP-16.urdf.xacro"/-->
+<xacro:include filename="$(find orne_description)/urdf/sensors/vlp16.urdf.xacro"/>
 <xacro:VLP-16 name="velodyne" parent="base_link">
     <origin xyz="0.098 0.0 0.422" rpy="0 0 -0.12"/>

File: orne_description/urdf/orne_alpha_sim.xacro (robot description, xacro)
@@ -7,6 +7,4 @@
 <xacro:include filename="$(find orne_description)/urdf/orne_x.xacro"/>
 <xacro:include filename="$(find icart_mini_description)/urdf/sensors/imu.urdf.xacro"/>
-<xacro:include filename="$(find icart_mini_description)/urdf/sensors/hokuyo.urdf.xacro"/>
-<xacro:include filename="$(find velodyne_description)/urdf/VLP-16.urdf.xacro"/>
 <!-- Setting for imu -->
 <xacro:sensor_imu name="imu" parent="base_link" size="0.05 0.05 0.05">
@@ -14,4 +12,5 @@
 </xacro:sensor_imu>
 <!-- Setting for levelly fixed 2D URG -->
+<xacro:include filename="$(find icart_mini_description)/urdf/sensors/hokuyo.urdf.xacro"/>
 <xacro:sensor_hokuyo name="hokuyo" parent="base_link">
     <origin xyz="0.212 0 0.2485" rpy="0 0 0"/>
@@ -30,7 +29,10 @@
 </xacro:sensor_hokuyo3d>
 -->
-<xacro:include filename="$(find velodyne_description)/urdf/VLP-16.urdf.xacro"/>
-<xacro:VLP-16 name="velodyne" parent="base_link">
+<xacro:include filename="$(find orne_description)/urdf/sensors/vlp16.urdf.xacro"/>
+<xacro:vlp16_2d name="velodyne" parent="base_link">
     <origin xyz="0.098 0.0 0.422" rpy="0 0 0"/>
-</xacro:VLP-16>
+</xacro:vlp16_2d>
+<xacro:vlp16_3d name="velodyne3d" parent="base_link">
+    <origin xyz="0.098 0.0 0.422" rpy="0 0 0"/>
+</xacro:vlp16_3d>
 </robot>

File: orne_description/urdf/orne_x.xacro (robot description, xacro)
@@ -25,5 +25,5 @@
       <origin xyz="0.005 0 0.305" rpy="0 0 0"/>
       <geometry>
-	       <box size=".376 .45 .242"/>
+	       <box size=".376 .45 .134"/>
       </geometry>
     </collision>
@@ -31,5 +31,5 @@
       <origin xyz="0.005 0 0.305" rpy="0 0 0"/>
       <geometry>
-	       <box size=".376 .45 .242"/>
+	       <box size=".376 .45 .134"/>
       </geometry>
       <material name="orange"/>
