Commit message: make real beta can nav with 2 urg

File: orne_description/urdf/orne_beta_2urg.xacro (robot description, xacro)
@@ -13,4 +13,7 @@
     <origin xyz="-0.34 0 0.22" rpy="0 0 3.1415927"/>
 </xacro:sensor_hokuyo>
+<xacro:sensor_hokuyo name="hokuyo_mid" parent="base_link">
+    <origin xyz="-0.07 0 0.22" rpy="0 0 0"/>
+</xacro:sensor_hokuyo>
 <xacro:include filename="$(find icart_mini_description)/urdf/sensors/hokuyo3d.urdf.xacro"/>
 <xacro:sensor_hokuyo3d name="hokuyo3d" parent="base_link">

Commit message: push

File: orne_description/urdf/orne_beta_2urg.xacro (robot description, xacro)
@@ -8,8 +8,8 @@
 <xacro:include filename="$(find icart_mini_description)/urdf/sensors/hokuyo.urdf.xacro"/>
 <xacro:sensor_hokuyo name="hokuyo" parent="base_link">
-    <origin xyz="0.2 0 0.22" rpy="0 0 0"/>
+    <origin xyz="0.098 0 0.422" rpy="0 0 0"/>
 </xacro:sensor_hokuyo>
 <xacro:sensor_hokuyo name="hokuyo_back" parent="base_link">
-    <origin xyz="-0.34 0 0.22" rpy="0 0 3.1415927"/>
+    <origin xyz="-0.042 0 0.422" rpy="0 0 3.1415927"/>
 </xacro:sensor_hokuyo>
 <xacro:sensor_hokuyo name="hokuyo_mid" parent="base_link">
