Commit message: Fixed imu link position

File: orne_description/urdf/orne_beta.xacro (robot description, xacro)
@@ -5,5 +5,5 @@
 <xacro:include filename="$(find icart_mini_description)/urdf/sensors/imu.urdf.xacro"/>
 <xacro:sensor_imu name="imu" parent="base_link">
-    <origin xyz="-0.18 0.0 0.170" rpy="0 0 0"/>
+    <origin xyz="0.19 0.0 0.15" rpy="0 0 0"/>
 </xacro:sensor_imu>
 </robot>

Commit message: change orne_middle to orne_beta

File: orne_description/urdf/orne_beta.xacro (robot description, xacro)
@@ -1,5 +1,5 @@
 <?xml version="1.0"?>
 <robot name="orne_beta" xmlns:xacro="http://www.ros.org/wiki/xacro">
-<xacro:include filename="$(find icart_mini_description)/urdf/icart_mini.xacro"/>
+<xacro:include filename="$(find orne_description)/urdf/icart_middle.xacro"/>
 <xacro:include filename="$(find icart_mini_description)/urdf/sensors/imu.urdf.xacro"/>
 <xacro:sensor_imu name="imu" parent="base_link" size="0.05 0.05 0.05">
@@ -8,5 +8,5 @@
 <xacro:include filename="$(find icart_mini_description)/urdf/sensors/hokuyo.urdf.xacro"/>
 <xacro:sensor_hokuyo name="hokuyo" parent="base_link">
-    <origin xyz="0.243 0 0.2" rpy="0 0 0"/>
+    <origin xyz="0.20 0 0.220" rpy="0 0 0"/>
 </xacro:sensor_hokuyo>
 </robot>

Commit message: respond to changes icart_mini.xacor

File: orne_description/urdf/orne_beta.xacro (robot description, xacro)
@@ -4,9 +4,9 @@
 <xacro:include filename="$(find icart_mini_description)/urdf/sensors/imu.urdf.xacro"/>
 <xacro:sensor_imu name="imu" parent="base_link" size="0.05 0.05 0.05">
-    <origin xyz="0.19 0.0 0.15" rpy="0 0 0"/>
+    <origin xyz="0.04 0.0 0.15" rpy="0 0 0"/>
 </xacro:sensor_imu>
 <xacro:include filename="$(find icart_mini_description)/urdf/sensors/hokuyo.urdf.xacro"/>
 <xacro:sensor_hokuyo name="hokuyo" parent="base_link">
-    <origin xyz="0.243 0 0.2" rpy="0 0 0"/>
+    <origin xyz="0.093 0 0.2" rpy="0 0 0"/>
 </xacro:sensor_hokuyo>
 </robot>

Commit message: fix orne_beta.xacro and rename launch name

File: orne_description/urdf/orne_beta.xacro (robot description, xacro)
@@ -8,5 +8,5 @@
 <xacro:include filename="$(find icart_mini_description)/urdf/sensors/hokuyo.urdf.xacro"/>
 <xacro:sensor_hokuyo name="hokuyo" parent="base_link">
-    <origin xyz="0.2 0 0.2" rpy="0 0 0"/>
+    <origin xyz="0.2 0 0.22" rpy="0 0 0"/>
 </xacro:sensor_hokuyo>
 </robot>

Commit message: add 3durg parameter to orne_beta.xacro

File: orne_description/urdf/orne_beta.xacro (robot description, xacro)
@@ -10,3 +10,7 @@
     <origin xyz="0.2 0 0.22" rpy="0 0 0"/>
 </xacro:sensor_hokuyo>
+<xacro:include filename="$(find icart_mini_description)/urdf/sensors/hokuyo3d.urdf.xacro"/>
+<xacro:sensor_hokuyo3d name="hokuyo3d" parent="base_link">
+    <origin xyz="0.12 0 0.50" rpy="3.14 -0.227 0.0"/>
+</xacro:sensor_hokuyo3d>
 </robot>

Commit message: Fix IMU yaw orientation

File: orne_description/urdf/orne_beta.xacro (robot description, xacro)
@@ -4,5 +4,5 @@
 <xacro:include filename="$(find icart_mini_description)/urdf/sensors/imu.urdf.xacro"/>
 <xacro:sensor_imu name="imu" parent="base_link" size="0.05 0.05 0.05">
-    <origin xyz="0.04 0.0 0.15" rpy="0 0 0"/>
+    <origin xyz="0.04 0.0 0.15" rpy="0 0 3.14"/>
 </xacro:sensor_imu>
 <xacro:include filename="$(find icart_mini_description)/urdf/sensors/hokuyo.urdf.xacro"/>

Commit message: add kinect v2

File: orne_description/urdf/orne_beta.xacro (robot description, xacro)
@@ -14,3 +14,7 @@
     <origin xyz="0.12 0 0.50" rpy="3.14 -0.227 0.0"/>
 </xacro:sensor_hokuyo3d>
+<xacro:include filename="$(find orne_description)/urdf/kinect_v2.urdf.xacro"/>
+<xacro:sensor_kinect_v2 name="kinect_v2" parent="base_link">
+    <origin xyz="0.12 0 0.60" rpy="0.0 0.0 0.0"/>
+</xacro:sensor_kinect_v2>
 </robot>

Commit message: 3D URGの位置変更

File: orne_description/urdf/orne_beta.xacro (robot description, xacro)
@@ -12,5 +12,5 @@
 <xacro:include filename="$(find icart_mini_description)/urdf/sensors/hokuyo3d.urdf.xacro"/>
 <xacro:sensor_hokuyo3d name="hokuyo3d" parent="base_link">
-    <origin xyz="0.12 0 0.50" rpy="3.14 -0.227 0.0"/>
+    <origin xyz="0.2 0 0.39" rpy="0.0 0.0 0.0"/>
 </xacro:sensor_hokuyo3d>
 </robot>

Commit message: hokuyo3dの角度変更

File: orne_description/urdf/orne_beta.xacro (robot description, xacro)
@@ -12,5 +12,5 @@
 <xacro:include filename="$(find icart_mini_description)/urdf/sensors/hokuyo3d.urdf.xacro"/>
 <xacro:sensor_hokuyo3d name="hokuyo3d" parent="base_link">
-    <origin xyz="0.2 0 0.39" rpy="0.0 0.0 0.0"/>
+    <origin xyz="0.2 0 0.39" rpy="0.0 0.21 0.0"/>
 </xacro:sensor_hokuyo3d>
 </robot>

Commit message: Update orne_beta.xacro

File: orne_description/urdf/orne_beta.xacro (robot description, xacro)
@@ -4,5 +4,5 @@
 <xacro:include filename="$(find icart_mini_description)/urdf/sensors/imu.urdf.xacro"/>
 <xacro:sensor_imu name="imu" parent="base_link" size="0.05 0.05 0.05">
-    <origin xyz="0.04 0.0 0.15" rpy="0 0 3.14"/>
+    <origin xyz="0.04 0.0 0.15" rpy="0 0 0"/>
 </xacro:sensor_imu>
 <xacro:include filename="$(find icart_mini_description)/urdf/sensors/hokuyo.urdf.xacro"/>

Commit message: IMU用にβのセンサの角度と起動launchファイルの変更

File: orne_description/urdf/orne_beta.xacro (robot description, xacro)
@@ -4,5 +4,5 @@
 <xacro:include filename="$(find icart_mini_description)/urdf/sensors/imu.urdf.xacro"/>
 <xacro:sensor_imu name="imu" parent="base_link" size="0.05 0.05 0.05">
-    <origin xyz="0.04 0.0 0.15" rpy="0 0 0"/>
+    <origin xyz="0.04 0.0 0.15" rpy="0 0 "/>
 </xacro:sensor_imu>
 <xacro:include filename="$(find icart_mini_description)/urdf/sensors/hokuyo.urdf.xacro"/>

Commit message: IMU用にβのセンサの角度と起動launchファイルの変更

File: orne_description/urdf/orne_beta.xacro (robot description, xacro)
@@ -4,5 +4,5 @@
 <xacro:include filename="$(find icart_mini_description)/urdf/sensors/imu.urdf.xacro"/>
 <xacro:sensor_imu name="imu" parent="base_link" size="0.05 0.05 0.05">
-    <origin xyz="0.04 0.0 0.15" rpy="0 0 "/>
+    <origin xyz="0.04 0.0 0.15" rpy="0 0 0"/>
 </xacro:sensor_imu>
 <xacro:include filename="$(find icart_mini_description)/urdf/sensors/hokuyo.urdf.xacro"/>

Commit message: chanage hokuyo3d rpy

File: orne_description/urdf/orne_beta.xacro (robot description, xacro)
@@ -12,5 +12,5 @@
 <xacro:include filename="$(find icart_mini_description)/urdf/sensors/hokuyo3d.urdf.xacro"/>
 <xacro:sensor_hokuyo3d name="hokuyo3d" parent="base_link">
-    <origin xyz="0.2 0 0.39" rpy="0.0 0.0 0.0"/>
+    <origin xyz="0.2 0 0.39" rpy="0.0 0.314 0.0"/>
 </xacro:sensor_hokuyo3d>
 </robot>

Commit message: revert parameters

File: orne_description/urdf/orne_beta.xacro (robot description, xacro)
@@ -12,5 +12,5 @@
 <xacro:include filename="$(find icart_mini_description)/urdf/sensors/hokuyo3d.urdf.xacro"/>
 <xacro:sensor_hokuyo3d name="hokuyo3d" parent="base_link">
-    <origin xyz="0.2 0 0.39" rpy="0.0 0.314 0.0"/>
+    <origin xyz="0.2 0 0.39" rpy="0.0 0.0 0.0"/>
 </xacro:sensor_hokuyo3d>
 </robot>

File: orne_description/urdf/sensors/vlp16.urdf.xacro (robot description, xacro)
@@ -64,4 +64,5 @@
           <scan>
             <horizontal>
+<!--          <samples>720</samples>  -->
               <samples>721</samples>
               <resolution>1.0</resolution>
