Commit message: detect obstacle

File: orne_description/urdf/orne_gamma.xacro (robot description, xacro)
@@ -1,8 +1,8 @@
 <?xml version="1.0"?>
 <robot name="orne_gamma" xmlns:xacro="http://www.ros.org/wiki/xacro">
-<xacro:include filename="$(find icart_mini_description)/urdf/icart_mini.xacro"/>
-<xacro:include filename="$(find icart_mini_description)/urdf/sensors/hokuyo.urdf.xacro"/>
-<xacro:sensor_hokuyo name="hokuyo" parent="base_link">
-    <origin xyz="0.2 0 0.1" rpy="0 0 0"/>
-</xacro:sensor_hokuyo>
+    <xacro:include filename="$(find icart_mini_description)/urdf/icart_mini.xacro"/>
+    <xacro:include filename="$(find icart_mini_description)/urdf/sensors/hokuyo.urdf.xacro"/>
+    <xacro:sensor_hokuyo name="hokuyo" parent="base_link">
+        <origin xyz="0.2 0 0.2" rpy="0 0 0"/>
+    </xacro:sensor_hokuyo>
 </robot>

Commit message: adjust sensor height

File: orne_description/urdf/orne_gamma.xacro (robot description, xacro)
@@ -10,5 +10,5 @@
 <xacro:include filename="$(find icart_mini_description)/urdf/sensors/hokuyo.urdf.xacro"/>
 <xacro:sensor_hokuyo name="hokuyo" parent="base_link">
-    <origin xyz="0.2 0 0.1" rpy="0 0 0"/>
+    <origin xyz="0.2 0 0.2" rpy="0 0 0"/>
 </xacro:sensor_hokuyo>
 </robot>
