Commit message: fix orne_X urdf

File: orne_description/urdf/orne_x.xacro (robot description, xacro)
@@ -12,29 +12,29 @@
       <origin xyz="0 0 0.1" rpy="0 0 0"/>
       <geometry>
-	<box size=".40 .45 .134"/>
+	       <box size=".40 .45 .134"/>
       </geometry>
     </collision>
     <visual>
-      <origin xyz="0 0 0.1" rpy="0 0 0"/>
+      <origin xyz="0.1 0 0.1" rpy="0 0 0"/>
       <geometry>
-	<box size=".40 .45 .134"/>
+	       <box size=".40 .45 .134"/>
       </geometry>
       <material name="orange"/>
     </visual>
     <collision>
-      <origin xyz="-0.095 0 0.305" rpy="0 0 0"/>
+      <origin xyz="0.005 0 0.305" rpy="0 0 0"/>
       <geometry>
-	<box size=".376 .45 .242"/>
+	       <box size=".376 .45 .242"/>
       </geometry>
     </collision>
     <visual>
-      <origin xyz="-0.095 0 0.305" rpy="0 0 0"/>
+      <origin xyz="0.005 0 0.305" rpy="0 0 0"/>
       <geometry>
-	<box size=".376 .45 .242"/>
+	       <box size=".376 .45 .242"/>
       </geometry>
       <material name="orange"/>
     </visual>
     <collision name="collision">
-      <origin xyz="0.201 -0.141 0.075" rpy="0 1.5707 1.5707"/>
+      <origin xyz="0.301 -0.141 0.075" rpy="0 1.5707 1.5707"/>
       <geometry>
         <cylinder  length="0.03" radius="0.075"/>
@@ -42,5 +42,5 @@
     </collision>
     <visual name="visual">
-      <origin xyz="0.201 -0.141 0.075" rpy="0 1.5707 1.5707"/>
+      <origin xyz="0.301 -0.141 0.075" rpy="0 1.5707 1.5707"/>
       <geometry>
         <cylinder  length="0.03" radius="0.075"/>
@@ -48,5 +48,5 @@
     </visual>
     <collision name="collision">
-      <origin xyz="0.201 0.141 0.075" rpy="0 1.5707 1.5707"/>
+      <origin xyz="0.301 0.141 0.075" rpy="0 1.5707 1.5707"/>
       <geometry>
         <cylinder  length="0.03" radius="0.075"/>
@@ -54,5 +54,5 @@
     </collision>
     <visual name="visual">
-      <origin xyz="0.201 0.141 0.075" rpy="0 1.5707 1.5707"/>
+      <origin xyz="0.301 0.141 0.075" rpy="0 1.5707 1.5707"/>
       <geometry>
         <cylinder  length="0.03" radius="0.075"/>
@@ -74,5 +74,5 @@
   </link>
   <joint type="fixed" name="visual_left_wheel_hinge">
-    <origin xyz="-0.145 0.233 0.15" rpy="0 0 0"/>
+    <origin xyz="-0.045 0.233 0.1518" rpy="0 0 0"/>
     <child link="visual_left_wheel">visual_left_wheel</child>
     <parent link="base_link">base_link</parent>
@@ -89,5 +89,5 @@
       <origin xyz="0 0.0 0" rpy="0 1.5707 1.5707"/>
       <geometry>
-        <cylinder  length="0.03" radius="0.151"/>
+        <cylinder  length="0.03" radius="0.0725"/>
       </geometry>
     </visual-->
@@ -99,5 +99,5 @@
   </link>
   <joint type="revolute" name="left_wheel_hinge">
-    <origin xyz="-0.145 0.223 0.15" rpy="0 0 0"/>
+    <origin xyz="-0.045 0.223 0.1518" rpy="0 0 0"/>
     <child link="left_wheel">left_wheel</child>
     <parent link="base_link">base_link</parent>
@@ -114,5 +114,5 @@
   </link>
   <joint type="fixed" name="visual_right_wheel_hinge">
-    <origin xyz="-0.145 -0.223 0.15" rpy="0 0 0"/>
+    <origin xyz="-0.045 -0.223 0.1518" rpy="0 0 0"/>
     <child link="visual_right_wheel">visual_right_wheel</child>
     <parent link="base_link">base_link</parent>
@@ -129,5 +129,5 @@
       <origin xyz="0 0.0 0" rpy="0 1.5707 1.5707"/>
       <geometry>
-        <cylinder  length="0.03" radius="0.151"/>
+        <cylinder  length="0.03" radius="0.0725"/>
       </geometry>
     </visual-->
@@ -135,9 +135,9 @@
       <mass value="1" />
       <origin xyz="0 0.0 0"/>
-      <inertia ixx="0.1" ixy="0" ixz="0" iyy="0.1" iyz="0" izz="1" />
+      <inertia ixx="0.1" ixy="0" ixz="0" iyy="0.1" iyz="0" izz="0.1" />
     </inertial>
   </link>
   <joint type="revolute" name="right_wheel_hinge">
-    <origin xyz="-0.145 -0.223 0.15" rpy="0 0 0"/>
+    <origin xyz="-0.045 -0.223 0.1518" rpy="0 0 0"/>
     <child link="right_wheel">right_wheel</child>
     <parent link="base_link">base_link</parent>

Commit message: fix sim bag for alpha

File: orne_description/urdf/orne_x.xacro (robot description, xacro)
@@ -36,5 +36,5 @@
     </visual>
     <collision name="collision">
-      <origin xyz="0.301 -0.141 0.075" rpy="1.57 0 0"/>
+      <origin xyz="0.301 -0.141 0.075" rpy="0 1.5707 1.5707"/>
       <geometry>
         <cylinder  length="0.03" radius="0.075"/>
@@ -42,5 +42,5 @@
     </collision>
     <visual name="visual">
-      <origin xyz="0.301 -0.141 0.075" rpy="1.57 0 0"/>
+      <origin xyz="0.301 -0.141 0.075" rpy="0 1.5707 1.5707"/>
       <geometry>
         <cylinder  length="0.03" radius="0.075"/>
@@ -48,5 +48,5 @@
     </visual>
     <collision name="collision">
-      <origin xyz="0.301 0.141 0.075" rpy="1.57 0 0"/>
+      <origin xyz="0.301 0.141 0.075" rpy="0 1.5707 1.5707"/>
       <geometry>
         <cylinder  length="0.03" radius="0.075"/>
@@ -54,5 +54,5 @@
     </collision>
     <visual name="visual">
-      <origin xyz="0.301 0.141 0.075" rpy="1.57 0 0"/>
+      <origin xyz="0.301 0.141 0.075" rpy="0 1.5707 1.5707"/>
       <geometry>
         <cylinder  length="0.03" radius="0.075"/>
@@ -67,5 +67,5 @@
   <link name="visual_left_wheel">
     <visual name="visual">
-      <origin xyz="0 0.0 0" rpy="1.57 0 0"/>
+      <origin xyz="0 0.0 0" rpy="0 1.5707 1.5707"/>
       <geometry>
         <cylinder  length="0.03" radius="0.151"/>
@@ -81,5 +81,5 @@
   <link name="left_wheel">
     <collision name="collision">
-      <origin xyz="0 0.0 0" rpy="1.57 0 0"/>
+      <origin xyz="0 0.0 0" rpy="0 1.5707 1.5707"/>
       <geometry>
          <cylinder  length="0.03" radius="0.151"/>
@@ -87,5 +87,5 @@
     </collision>
     <!--visual name="visual">
-      <origin xyz="0 0.0 0" rpy="0 0 0"/>
+      <origin xyz="0 0.0 0" rpy="0 1.5707 1.5707"/>
       <geometry>
         <cylinder  length="0.03" radius="0.0725"/>
@@ -107,5 +107,5 @@
   <link name="visual_right_wheel">
     <visual name="visual">
-      <origin xyz="0 0.0 0" rpy="1.57 0 0"/>
+      <origin xyz="0 0.0 0" rpy="0 1.5707 1.5707"/>
       <geometry>
         <cylinder  length="0.03" radius="0.151"/>
@@ -121,5 +121,5 @@
   <link name="right_wheel">
     <collision name="collision">
-      <origin xyz="0 0.0 0" rpy="1.57 00 00"/>
+      <origin xyz="0 0.0 0" rpy="0 1.5707 1.5707"/>
       <geometry>
          <cylinder  length="0.03" radius="0.151"/>
@@ -127,5 +127,5 @@
     </collision>
     <!--visual name="visual">
-      <origin xyz="0 0.0 0" rpy="0 0 0"/>
+      <origin xyz="0 0.0 0" rpy="0 1.5707 1.5707"/>
       <geometry>
         <cylinder  length="0.03" radius="0.0725"/>

Commit message: change

File: orne_description/urdf/orne_x.xacro (robot description, xacro)
@@ -60,5 +60,5 @@
     </visual>
     <inertial>
-       <mass value="15" />
+       <mass value="150" />
        <origin xyz="0 0 0" rpy="0 0 0"/>
        <inertia ixx="1" ixy="0" ixz="0" iyy="1" iyz="0" izz="1" />

Commit message: revert kinetic's parameter

File: orne_description/urdf/orne_x.xacro (robot description, xacro)
@@ -60,5 +60,5 @@
     </visual>
     <inertial>
-       <mass value="150" />
+       <mass value="15" />
        <origin xyz="0 0 0" rpy="0 0 0"/>
        <inertia ixx="1" ixy="0" ixz="0" iyy="1" iyz="0" izz="1" />

Commit message: add base_footprint

File: orne_description/urdf/orne_x.xacro (robot description, xacro)
@@ -7,4 +7,11 @@
   <xacro:include filename="$(find icart_mini_description)/urdf/materials.xacro" />
   <xacro:include filename="$(find orne_description)/urdf/orne_x.gazebo"/>
+ <!-- Base footprint-->
+ <link name="base_footprint"/>
+  <joint name="base_joint" type="fixed">
+    <parent link="base_footprint"/>
+    <child link="base_link"/>
+    <origin xyz="0.0 0.0 0.010" rpy="0 0 0"/>
+  </joint>
   <!-- Base Link -->
   <link name="base_link">
