Commit message: add_gnss

File: orne_description/urdf/orne_alpha_sim.xacro (robot description, xacro)
@@ -31,5 +31,5 @@
 <xacro:include filename="$(find orne_description)/urdf/sensors/vlp16.urdf.xacro"/>
 <xacro:vlp16_2d name="velodyne" parent="base_link">
-    <origin xyz="0.098 0.0 0.422" rpy="0 0 0"/>
+    <origin xyz="zz 0.0 0.422" rpy="0 0 0"/>
 </xacro:vlp16_2d>
 <!--

File: orne_description/urdf/orne_alpha_with_vision_sim.xacro (robot description, xacro)
@@ -7,9 +7,7 @@
 <xacro:include filename="$(find orne_description)/urdf/orne_x.xacro"/>
 <xacro:include filename="$(find icart_mini_description)/urdf/sensors/imu.urdf.xacro"/>
-<!-- Setting for imu -->
 <xacro:sensor_imu name="imu" parent="base_link" size="0.05 0.05 0.05">
     <origin xyz="-0.145 0.0 0.21" rpy="0 0 0"/>
 </xacro:sensor_imu>
-<!-- Setting for levelly fixed 2D URG -->
 <xacro:include filename="$(find icart_mini_description)/urdf/sensors/hokuyo.urdf.xacro"/>
 <xacro:sensor_hokuyo name="hokuyo" parent="base_link">
@@ -31,5 +29,5 @@
 <xacro:include filename="$(find orne_description)/urdf/sensors/vlp16.urdf.xacro"/>
 <xacro:vlp16_2d name="velodyne" parent="base_link">
-    <origin xyz="0.098 0.0 0.422" rpy="0 0 0"/>
+    <origin xyz="1 1 1" rpy="0 0 0"/>
 </xacro:vlp16_2d>
 <!--
@@ -39,6 +37,9 @@
 -->
 <!-- Setting for camera -->
-    <xacro:include filename="$(find orne_description)/urdf/sensors/camera.urdf.xacro"/>
-    <xacro:usb_camera prefix="camera"/>
+<xacro:include filename="$(find orne_description)/urdf/sensors/camera.urdf.xacro"/>
+<xacro:usb_camera prefix="camera"/>
+<!-- Setting fot gps -->
+<xacro:include filename="$(find orne_description)/urdf/sensors/gps.urdf.xacro"/>
+<xacro:gps prefix="gps"/>
   <gazebo>
     <plugin name="ground_truth" filename="libgazebo_ros_p3d.so">

File: orne_description/urdf/sensors/camera.urdf.xacro (robot description, xacro)
@@ -39,6 +39,6 @@
                     <horizontal_fov>1.3962634</horizontal_fov>
                     <image>
-                        <width>1280</width>
-                        <height>720</height>
+                        <width>640</width>
+                        <height>480</height>
                         <format>R8G8B8</format>
                     </image>
