Commit message: VLP16のパラメータ変更

File: orne_description/urdf/sensors/vlp16.urdf.xacro (robot description, xacro)
@@ -31,29 +31,29 @@
   </xacro:macro>
   <xacro:macro name="vlp16_2d" params="name parent *origin">
-	  <joint name="${name}_joint" type="fixed">
-	      <axis xyz="1 0 0"/>
-	      <insert_block name="origin"/>
-	      <parent link="${parent}"/>
-	      <child link="${name}"/>
-	  </joint>
-	  <link name="${name}">
-	      <inertial>
-	        <mass value="0.001"/>
-	        <origin rpy="0 0 0" xyz="0 0 0"/>
-	        <inertia ixx="0.0001" ixy="0" ixz="0" iyy="0.000001" iyz="0" izz="0.0001"/>
-	      </inertial>
-	      <visual>
-	        <origin rpy="0 0 0.1" xyz="0 0 0"/>
-	        <geometry>
-	          <box size="0.1 0.1 0.1"/>
-	        </geometry>
-	      </visual>
-	      <collision>
-	        <origin rpy="0 0 0.1" xyz="0 0 0"/>
-	        <geometry>
-	          <box size="0.1 0.1 0.1"/>
-	        </geometry>
-	      </collision>
-	  </link>
+    <joint name="${name}_joint" type="fixed">
+        <axis xyz="1 0 0"/>
+        <insert_block name="origin"/>
+        <parent link="${parent}"/>
+        <child link="${name}"/>
+    </joint>
+    <link name="${name}">
+        <inertial>
+          <mass value="0.001"/>
+          <origin rpy="0 0 0" xyz="0 0 0"/>
+          <inertia ixx="0.0001" ixy="0" ixz="0" iyy="0.000001" iyz="0" izz="0.0001"/>
+        </inertial>
+        <visual>
+          <origin rpy="0 0 0.1" xyz="0 0 0"/>
+          <geometry>
+            <box size="0.1 0.1 0.1"/>
+          </geometry>
+        </visual>
+        <collision>
+          <origin rpy="0 0 0.1" xyz="0 0 0"/>
+          <geometry>
+            <box size="0.1 0.1 0.1"/>
+          </geometry>
+        </collision>
+    </link>
       <gazebo reference="${name}">
         <sensor name="velodyne_2d" type="ray">
@@ -71,5 +71,5 @@
           </scan>
           <range>
-            <min>0.90</min>
+            <min>0.10</min>
             <max>100.0</max>
             <resolution>0.01</resolution>
@@ -89,29 +89,29 @@
   </xacro:macro>
   <xacro:macro name="vlp16_3d" params="name parent *origin">
-	  <joint name="${name}_joint" type="fixed">
-	      <axis xyz="1 0 0"/>
-	      <insert_block name="origin"/>
-	      <parent link="${parent}"/>
-	      <child link="${name}"/>
-	  </joint>
-	  <link name="${name}">
-	      <inertial>
-	        <mass value="0.001"/>
-	        <origin rpy="0 0 0" xyz="0 0 0"/>
-	        <inertia ixx="0.0001" ixy="0" ixz="0" iyy="0.000001" iyz="0" izz="0.0001"/>
-	      </inertial>
-	      <visual>
-	        <origin rpy="0 0 0.1" xyz="0 0 0"/>
-	        <geometry>
-	          <box size="0.1 0.1 0.1"/>
-	        </geometry>
-	      </visual>
-	      <collision>
-	        <origin rpy="0 0 0.1" xyz="0 0 0"/>
-	        <geometry>
-	          <box size="0.1 0.1 0.1"/>
-	        </geometry>
-	      </collision>
-	  </link>
+    <joint name="${name}_joint" type="fixed">
+        <axis xyz="1 0 0"/>
+        <insert_block name="origin"/>
+        <parent link="${parent}"/>
+        <child link="${name}"/>
+    </joint>
+    <link name="${name}">
+        <inertial>
+          <mass value="0.001"/>
+          <origin rpy="0 0 0" xyz="0 0 0"/>
+        <inertia ixx="0.0001" ixy="0" ixz="0" iyy="0.000001" iyz="0" izz="0.0001"/>
+        </inertial>
+        <visual>
+          <origin rpy="0 0 0.1" xyz="0 0 0"/>
+          <geometry>
+            <box size="0.1 0.1 0.1"/>
+          </geometry>
+       </visual>
+       <collision>
+          <origin rpy="0 0 0.1" xyz="0 0 0"/>
+          <geometry>
+            <box size="0.1 0.1 0.1"/>
+          </geometry>
+        </collision>
+    </link>
     <gazebo reference="${name}">
       <sensor name="velodyne_3d" type="ray">
@@ -122,5 +122,5 @@
         <scan>
           <horizontal>
-            <samples>145</samples>
+            <samples>1825</samples>
             <resolution>1.0</resolution>
             <min_angle>-3.141592</min_angle>
@@ -130,10 +130,10 @@
             <samples>16</samples>
             <resolution>1.0</resolution>
-            <min_angle>-0.0872664626</min_angle>
-            <max_angle>0.610865238</max_angle>
+            <min_angle>-0.2617993875</min_angle>
+            <max_angle>0.2617993875</max_angle>
           </vertical>
         </scan>
         <range>
-          <min>0.90</min>
+          <min>0.10</min>
           <max>100.0</max>
           <resolution>0.01</resolution>

Commit message: レンジの修正

File: orne_description/urdf/sensors/vlp16.urdf.xacro (robot description, xacro)
@@ -19,5 +19,5 @@
             <origin rpy="0 0 0.1" xyz="0 0 0"/>
             <geometry>
-              <box size="0.1 0.1 0.1"/>
+              <box size="0.05 0.05 0.05"/>
             </geometry>
           </visual>
@@ -25,5 +25,5 @@
             <origin rpy="0 0 0.1" xyz="0 0 0"/>
             <geometry>
-              <box size="0.1 0.1 0.1"/>
+              <box size="0.05 0.05 0.05"/>
             </geometry>
           </collision>
@@ -71,6 +71,6 @@
           </scan>
           <range>
-            <min>0.10</min>
-            <max>100.0</max>
+            <min>0.40</min>
+            <max>130.0</max>
             <resolution>0.01</resolution>
           </range>
@@ -135,6 +135,6 @@
         </scan>
         <range>
-          <min>0.10</min>
-          <max>100.0</max>
+          <min>0.40</min>
+          <max>130.0</max>
           <resolution>0.01</resolution>
         </range>

Commit message: fix: fix sensor position

File: orne_description/urdf/sensors/vlp16.urdf.xacro (robot description, xacro)
@@ -32,4 +32,5 @@
   <xacro:macro name="vlp16_2d" params="name parent *origin">
     <joint name="${name}_joint" type="fixed">
+        <origin xyz="0.098 0.0 0.422" rpy="0 0 0"/>
         <axis xyz="1 0 0"/>
         <insert_block name="origin"/>
