Commit message: refact gamma and alpha

File: orne_description/urdf/alpha/orne_alpha.urdf.xacro (robot description, xacro)
@@ -5,6 +5,15 @@
   <xacro:property name="PI" value="3.1415926535897931"/>
   <!-- Import Rviz colors -->
-  <xacro:include filename="$(find icart_mini_description)/urdf/materials.xacro" />
-  <xacro:include filename="$(find orne_description)/urdf/orne_x.gazebo"/>
+  <xacro:include filename="$(find orne_description)/urdf/material_colors.xacro" />
+  <xacro:include filename="$(find orne_description)/urdf/alpha/orne_alpha.gazebo"/>
+  <xacro:include filename="$(find orne_description)/urdf/sensors/imu.urdf.xacro"/>
+  <xacro:include filename="$(find orne_description)/urdf/sensors/hokuyo.urdf.xacro"/>
+  <!--Base footprint -->
+  <link name="base_footprint" />
+  <joint name="base_joint" type="fixed">
+    <origin xyz="0 0 0" />
+    <parent link="base_footprint" />
+    <child link="base_link" />
+  </joint>
   <!-- Base Link -->
   <link name="base_link">
@@ -65,4 +74,12 @@
     </inertial>
   </link>
+  <!-- Setting for imu -->
+  <xacro:sensor_imu name="imu" parent="base_link" size="0.05 0.05 0.05">
+      <origin xyz="-0.145 0.0 0.21" rpy="0 0 0"/>
+  </xacro:sensor_imu>
+  <!-- Setting for levelly fixed 2D URG -->
+  <xacro:sensor_hokuyo name="hokuyo" parent="base_link" size="0.05 0.05 0.05">
+      <origin xyz="0.212 0 0.2485" rpy="0 0 0"/>
+  </xacro:sensor_hokuyo>
   <link name="visual_left_wheel">
     <visual name="visual">

File: orne_description/urdf/alpha/orne_alpha_sim.xacro (robot description, xacro)
@@ -6,21 +6,26 @@
 >
 <xacro:include filename="$(find orne_description)/urdf/orne_x.xacro"/>
+<!-- <xacro:include filename="$(find orne_description)/urdf/orne_x.urdf"/> -->
 <xacro:include filename="$(find icart_mini_description)/urdf/sensors/imu.urdf.xacro"/>
-<xacro:include filename="$(find icart_mini_description)/urdf/sensors/hokuyo.urdf.xacro"/>
 <!-- Setting for imu -->
 <xacro:sensor_imu name="imu" parent="base_link" size="0.05 0.05 0.05">
-    <origin xyz="-0.145 0.0 0.21" rpy="0 3.14 0"/>
+    <origin xyz="-0.145 0.0 0.21" rpy="0 0 0"/>
 </xacro:sensor_imu>
+<!-- <joint name="hokuyo_joint" type="fixed">
+    <parent link="base_link"/>
+    <child link="hokuyo_link"/>
+    <origin xyz="0.212 0 0.2485" rpy="0 0 0"/>
+</joint>> -->
 <!-- Setting for levelly fixed 2D URG -->
+<!-- <xacro:include filename="$(find icart_mini_description)/urdf/sensors/hokuyo.urdf.xacro"/>
 <xacro:sensor_hokuyo name="hokuyo" parent="base_link">
     <origin xyz="0.212 0 0.2485" rpy="0 0 0"/>
-</xacro:sensor_hokuyo>
+    <origin xyz="0.0 0.0 0.0" rpy="0.0 0.0 0.0"/>
+</xacro:sensor_hokuyo> -->
 <!-- Setting for diagonally fixed 2D URG -->
-<!--
 <xacro:include filename="$(find icart_mini_description)/urdf/sensors/hokuyo.urdf.xacro"/>
 <xacro:sensor_hokuyo name="diagonally_hokuyo" parent="base_link">
    <origin xyz="0.098 0 0.422" rpy="0 0.296706 0"/>
 </xacro:sensor_hokuyo>
--->
 <!--
 <xacro:include filename="$(find icart_mini_description)/urdf/sensors/hokuyo3d.urdf.xacro"/>
@@ -29,8 +34,12 @@
 </xacro:sensor_hokuyo3d>
 -->
-<!--$acro:include filename="$(find velodyne_description)/urdf/VLP-16.urdf.xacro"/-->
 <xacro:include filename="$(find orne_description)/urdf/sensors/vlp16.urdf.xacro"/>
-<xacro:VLP-16 name="velodyne" parent="base_link">
-    <origin xyz="0.098 0.0 0.422" rpy="0 0 -0.12"/>
-</xacro:VLP-16>
+<xacro:vlp16_2d name="velodyne" parent="base_link">
+    <origin xyz="0.098 0.0 0.422" rpy="0 0 0"/>
+</xacro:vlp16_2d>
+<!--
+<xacro:vlp16_3d name="velodyne3d" parent="base_link">
+    <origin xyz="0.098 0.0 0.422" rpy="0 0 0"/>
+</xacro:vlp16_3d>
+-->
 </robot>

Commit message: fix urdf

File: orne_description/urdf/alpha/orne_alpha.urdf.xacro (robot description, xacro)
@@ -1,5 +1,5 @@
 <?xml version="1.0"?>
 <!-- Revolute-Revolute Manipulator -->
-<robot name="orne_x" xmlns:xacro="http://ros.org/wiki/xacro">
+<robot name="orne_alpha" xmlns:xacro="http://ros.org/wiki/xacro">
   <!-- Constants for robot dimensions -->
   <xacro:property name="PI" value="3.1415926535897931"/>
@@ -82,5 +82,5 @@
       <origin xyz="0.212 0 0.2485" rpy="0 0 0"/>
   </xacro:sensor_hokuyo>
-  <link name="visual_left_wheel">
+  <!-- <link name="visual_left_wheel">
     <visual name="visual">
       <origin xyz="0 0.0 0" rpy="0 1.5707 1.5707"/>
@@ -89,24 +89,26 @@
       </geometry>
     </visual>
-  </link>
-  <joint type="fixed" name="visual_left_wheel_hinge">
+  </link> -->
+  <!-- <joint type="fixed" name="visual_left_wheel_joint">
     <origin xyz="-0.045 0.233 0.1518" rpy="0 0 0"/>
     <child link="visual_left_wheel">visual_left_wheel</child>
     <parent link="base_link">base_link</parent>
     <axis xyz="0 1 0"/>
-  </joint>
+  </joint> -->
   <link name="left_wheel">
     <collision name="collision">
-      <origin xyz="0 0.0 0" rpy="0 1.5707 1.5707"/>
+      <!-- <origin xyz="0 0.0 0" rpy="0 1.5707 1.5707"/> -->
+      <origin xyz="0 0.0 0" rpy="0 0 0"/>
       <geometry>
          <cylinder  length="0.03" radius="0.151"/>
       </geometry>
     </collision>
-    <!--visual name="visual">
-      <origin xyz="0 0.0 0" rpy="0 1.5707 1.5707"/>
+    <visual name="visual">
+      <!-- <origin xyz="0 0.0 0" rpy="0 1.5707 1.5707"/> -->
+      <origin xyz="0 0.0 0" rpy="0 0 0"/>
       <geometry>
-        <cylinder  length="0.03" radius="0.0725"/>
+        <cylinder  length="0.03" radius="0.151"/>
       </geometry>
-    </visual-->
+    </visual>
     <inertial>
       <mass value="1" />
@@ -115,12 +117,12 @@
     </inertial>
   </link>
-  <joint type="revolute" name="left_wheel_hinge">
-    <origin xyz="-0.045 0.223 0.1518" rpy="0 0 0"/>
+  <joint type="revolute" name="left_wheel_joint">
+    <origin xyz="-0.045 0.223 0.1518" rpy="-1.57 0 0"/>
     <child link="left_wheel">left_wheel</child>
     <parent link="base_link">base_link</parent>
-    <axis xyz="0 1 0"/>
+    <axis xyz="0 0 1i"/>
     <limit effort="100" velocity="100.0"  lower="-5000" upper="5000" />
   </joint>
-  <link name="visual_right_wheel">
+  <!-- <link name="visual_right_wheel">
     <visual name="visual">
       <origin xyz="0 0.0 0" rpy="0 1.5707 1.5707"/>
@@ -129,24 +131,26 @@
       </geometry>
     </visual>
-  </link>
-  <joint type="fixed" name="visual_right_wheel_hinge">
+  </link> -->
+  <!-- <joint type="fixed" name="visual_right_wheel_joint">
     <origin xyz="-0.045 -0.223 0.1518" rpy="0 0 0"/>
     <child link="visual_right_wheel">visual_right_wheel</child>
     <parent link="base_link">base_link</parent>
     <axis xyz="0 1 0"/>
-  </joint>
+  </joint> -->
   <link name="right_wheel">
     <collision name="collision">
-      <origin xyz="0 0.0 0" rpy="0 1.5707 1.5707"/>
+      <!-- <origin xyz="0 0.0 0" rpy="0 1.5707 1.5707"/> -->
+      <origin xyz="0 0.0 0" rpy="0 0 0"/>
       <geometry>
          <cylinder  length="0.03" radius="0.151"/>
       </geometry>
     </collision>
-    <!--visual name="visual">
-      <origin xyz="0 0.0 0" rpy="0 1.5707 1.5707"/>
+    <visual name="visual">
+      <!-- <origin xyz="0 0.0 0" rpy="0 1.5707 1.5707"/> -->
+      <origin xyz="0 0.0 0" rpy="0 0 0"/>
       <geometry>
-        <cylinder  length="0.03" radius="0.0725"/>
+        <cylinder  length="0.03" radius="0.151"/>
       </geometry>
-    </visual-->
+    </visual>
     <inertial>
       <mass value="1" />
@@ -155,14 +159,14 @@
     </inertial>
   </link>
-  <joint type="revolute" name="right_wheel_hinge">
-    <origin xyz="-0.045 -0.223 0.1518" rpy="0 0 0"/>
+  <joint type="revolute" name="right_wheel_joint">
+    <origin xyz="-0.045 -0.223 0.1518" rpy="-1.57 0 0"/>
     <child link="right_wheel">right_wheel</child>
     <parent link="base_link">base_link</parent>
-    <axis xyz="0 1 0"/>
+    <axis xyz="0 0 1"/>
     <limit effort="100" velocity="100.0"  lower="-5000" upper="5000" />
   </joint>
   <transmission name="tran1">
     <type>transmission_interface/SimpleTransmission</type>
-    <joint name="left_wheel_hinge">
+    <joint name="left_wheel_joint">
       <hardwareInterface>VelocityJointInterface</hardwareInterface>
     </joint>
@@ -174,5 +178,5 @@
   <transmission name="tran2">
     <type>transmission_interface/SimpleTransmission</type>
-    <joint name="right_wheel_hinge">
+    <joint name="right_wheel_joint">
       <hardwareInterface>VelocityJointInterface</hardwareInterface>
     </joint>

File: orne_description/urdf/gamma/orne_gamma.urdf.xacro (robot description, xacro)
@@ -32,4 +32,16 @@
       </geometry>
     </collision>
+     <collision name="collision">
+      <origin xyz="0.15 0.0 -0.075" rpy="1.57 0.0 0.0"/>
+      <geometry>
+        <cylinder  length="0.03" radius="0.04625"/>
+      </geometry>
+    </collision>
+    <visual name="visual">
+      <origin xyz="0.15 0.0 -0.075" rpy="1.57 0.0 0.0"/>
+      <geometry>
+        <cylinder  length="0.03" radius="0.04625"/>
+      </geometry>
+    </visual>
     <inertial>
       <mass value="20" />
@@ -38,7 +50,7 @@
    </inertial>
  </link>
-   <link name="caster">
-    <collision name="collision">
-      <!-- <origin xyz="-0.325 0.0 0.05" rpy="0 1.5707 1.5707"/> -->
+   <!-- <link name="caster"> -->
+    <!-- <collision name="collision">
+      <origin xyz="0.15 0.0 -0.075" rpy="1.57 0.0 0.0"/>
       <geometry>
         <cylinder  length="0.03" radius="0.04625"/>
@@ -46,16 +58,16 @@
     </collision>
     <visual name="visual">
-      <!-- <origin xyz="-0.325 0.0 -0.075" rpy="0 1.5707 1.5707"/> -->
+      <origin xyz="-0.325 0.0 -0.075" rpy="0 1.5707 1.5707"/>
       <geometry>
         <cylinder  length="0.03" radius="0.04625"/>
       </geometry>
-    </visual>
-    </link>
-  <joint name="caster_joint" type="continuous">
+    </visual> -->
+    <!-- </link> -->
+  <!-- <joint name="caster_joint" type="continuous">
     <axis xyz="0 0 1"/>
     <parent link="base_link"/>
     <child link="caster"/>
     <origin xyz="0.15  0.0 -0.075" rpy="1.57 0 0"/>
-  </joint>
+  </joint> -->
   <!-- <link name="caster_support">
     <visual name="visual">
@@ -90,5 +102,5 @@
     <inertial>
       <mass value="1" />
-      <origin xyz="0.15 0.15 -0.05" rpy="1.57 0.0 0.0"/>
+      <origin xyz="-0.15 0.15 -0.05" rpy="-1.57 0.0 0.0"/>
       <inertia ixx="0.1" ixy="0" ixz="0" iyy="0.1" iyz="0" izz="0.1" />
     </inertial>
@@ -96,5 +108,5 @@
   <joint type="continuous" name="left_wheel_joint">
     <!-- <origin xyz="0 0.15 0.075" rpy="0 0 0"/> -->
-    <origin xyz="-0.15 0.15 -0.05" rpy="1.57 0 0"/>
+    <origin xyz="-0.15 0.15 -0.05" rpy="-1.57 0 0"/>
     <child link="left_wheel"></child>
     <parent link="base_link"></parent>
@@ -132,5 +144,5 @@
     <inertial>
       <mass value="1" />
-      <origin xyz="0 0.0 0"/>
+       <origin xyz="-0.15 0.15 -0.05" rpy="-1.57 0.0 0.0"/>
       <inertia ixx="0.1" ixy="0" ixz="0" iyy="0.1" iyz="0" izz="0.1" />
     </inertial>
@@ -139,5 +151,5 @@
     <!-- <origin xyz="0 -0.15 0.075" rpy="0 0 0"/> -->
     <!-- <origin xyz="0 0.0 -0.10" rpy="0 1.5707 1.5707"/> -->
-    <origin xyz="-0.15 -0.15 -0.05" rpy="1.57 0 0"/>
+    <origin xyz="-0.15 -0.15 -0.05" rpy="-1.57 0 0"/>
     <child link="right_wheel"></child>
     <parent link="base_link"></parent>

Commit message: separate param

File: orne_description/urdf/alpha/orne_alpha.urdf.xacro (robot description, xacro)
@@ -21,5 +21,5 @@
       <origin xyz="0 0 0.1" rpy="0 0 0"/>
       <geometry>
-	       <box size=".40 .45 .134"/>
+	       <box size=".40 .40 .134"/>
       </geometry>
     </collision>
@@ -27,5 +27,5 @@
       <origin xyz="0.1 0 0.1" rpy="0 0 0"/>
       <geometry>
-	       <box size=".40 .45 .134"/>
+	       <box size=".40 .40 .134"/>
       </geometry>
       <material name="orange"/>
@@ -34,5 +34,5 @@
       <origin xyz="0.005 0 0.305" rpy="0 0 0"/>
       <geometry>
-	       <box size=".376 .45 .134"/>
+	       <box size=".376 .40 .134"/>
       </geometry>
     </collision>
@@ -40,5 +40,5 @@
       <origin xyz="0.005 0 0.305" rpy="0 0 0"/>
       <geometry>
-	       <box size=".376 .45 .134"/>
+	       <box size=".376 .40 .134"/>
       </geometry>
       <material name="orange"/>
@@ -119,7 +119,7 @@
   <joint type="revolute" name="left_wheel_joint">
     <origin xyz="-0.045 0.223 0.1518" rpy="-1.57 0 0"/>
-    <child link="left_wheel">left_wheel</child>
-    <parent link="base_link">base_link</parent>
-    <axis xyz="0 0 1i"/>
+    <child link="left_wheel"></child>
+    <parent link="base_link"></parent>
+    <axis xyz="0 0 1"/>
     <limit effort="100" velocity="100.0"  lower="-5000" upper="5000" />
   </joint>
@@ -161,6 +161,6 @@
   <joint type="revolute" name="right_wheel_joint">
     <origin xyz="-0.045 -0.223 0.1518" rpy="-1.57 0 0"/>
-    <child link="right_wheel">right_wheel</child>
-    <parent link="base_link">base_link</parent>
+    <child link="right_wheel"></child>
+    <parent link="base_link"></parent>
     <axis xyz="0 0 1"/>
     <limit effort="100" velocity="100.0"  lower="-5000" upper="5000" />

File: orne_description/urdf/gamma/orne_gamma.urdf.xacro (robot description, xacro)
@@ -25,5 +25,5 @@
       <!-- <material name="orange"/> -->
     </visual>
-    <collision>
+    <collision name="collision">
       <!-- <origin xyz="-0.15 0 0.1" rpy="0 0 0"/> -->
       <origin xyz="0.0 0.0 0.0" rpy="0.0 0.0 0.0"/>>
@@ -44,9 +44,14 @@
       </geometry>
     </visual>
-    <inertial>
+    <!-- <inertial>
       <mass value="20" />
       <origin xyz="-0.08 0 0" rpy="0 0 0"/>
       <inertia ixx="1" ixy="0" ixz="0" iyy="1" iyz="0" izz="1" />
-   </inertial>
+   </inertial> -->
+   <inertial>
+    <mass value="15" />
+    <origin xyz="0 0 0" rpy="0 0 0"/>
+    <inertia ixx="1" ixy="0" ixz="0" iyy="1" iyz="0" izz="1" />
+    </inertial>
  </link>
    <!-- <link name="caster"> -->

File: orne_description/urdf/gamma/orne_gamma_caster.urdf.xacro (robot description, xacro)
@@ -7,4 +7,5 @@
   <xacro:include filename="$(find orne_box_description)/urdf/material_colors.xacro"/>
   <xacro:include filename="$(find orne_box_description)/urdf/sensors/hokuyo.urdf.xacro"/>
+  <xacro:include filename="$(find orne_description)/urdf/gamma/orne_gamma.gazebo"/>
   <!--Base Footprint-->
   <link name="base_footprint" />

File: orne_description/urdf/sensors/imu.urdf.xacro (robot description, xacro)
@@ -22,7 +22,7 @@
       </visual>
     </link>
-      <gazebo>
+      <!-- <gazebo>
         <plugin name="ros_imu" filename="libgazebo_ros_imu.so">
-          <bodyName>${parent}</bodyName> <!-- bodyName always set base_link by URDF parser -->
+          <bodyName>${parent}</bodyName>
           <topicName>imu_data</topicName>
           <serviceName>imu_service</serviceName>
@@ -32,4 +32,5 @@
         </plugin>
       </gazebo>
+    -->
   </xacro:macro>
 </robot>

Commit message: fix current tsukuba_ws

File: orne_description/urdf/alpha/orne_alpha.urdf.xacro (robot description, xacro)
@@ -32,5 +32,5 @@
     </visual>
     <collision>
-      <origin xyz="0.005 0 0.305" rpy="0 0 0"/>
+      <origin xyz="0.005 0 0.300" rpy="0 0 0"/>
       <geometry>
 	       <box size=".376 .40 .134"/>
@@ -80,5 +80,5 @@
   <!-- Setting for levelly fixed 2D URG -->
   <xacro:sensor_hokuyo name="hokuyo" parent="base_link" size="0.05 0.05 0.05">
-      <origin xyz="0.212 0 0.2485" rpy="0 0 0"/>
+      <origin xyz="0.212 0 0.375" rpy="0 0 0"/>
   </xacro:sensor_hokuyo>
   <!-- <link name="visual_left_wheel">
