Commit message: fix caster

File: orne_description/urdf/gamma/orne_gamma_caster.urdf.xacro (robot description, xacro)
@@ -1,171 +1,43 @@
 <?xml version="1.0"?>
-<!-- Revolute-Revolute Manipulator -->
-<robot name="orne_gamma" xmlns:xacro="http://www.ros.org/wiki/xacro">
-  <!-- Constants for robot dimensions -->
-  <xacro:property name="PI" value="3.1415926535897931"/>
-  <!-- Import Rviz colors -->
-  <xacro:include filename="$(find orne_box_description)/urdf/material_colors.xacro"/>
-  <xacro:include filename="$(find orne_box_description)/urdf/sensors/hokuyo.urdf.xacro"/>
-  <xacro:include filename="$(find orne_description)/urdf/gamma/orne_gamma.gazebo"/>
-  <!--Base Footprint-->
-  <link name="base_footprint" />
-  <joint name="base_joint" type="fixed">
-    <origin xyz="0 0 0" />
-    <parent link="base_footprint" />
-    <child link="base_link" />
-  </joint>
-  <!-- Base Link -->
-  <link name="base_link">
-    <visual>
-      <!-- <origin xyz="-0.15 0 0.1" rpy="0 0 0"/> -->
-      <origin xyz="0.0 0.0 0.0" rpy="0.0 0.0 0.0"/>>
-      <geometry>
-	    <box size=".485 .43 .15"/>
-      </geometry>
-      <!-- <material name="orange"/> -->
-    </visual>
-    <collision>
-      <!-- <origin xyz="-0.15 0 0.1" rpy="0 0 0"/> -->
-      <origin xyz="0.0 0.0 0.0" rpy="0.0 0.0 0.0"/>>
-      <geometry>
-	    <box size=".485 .43 .15"/>
-      </geometry>
-    </collision>
-    <inertial>
-      <mass value="10" />
-      <origin xyz="-0.08 0 0" rpy="0 0 0"/>
-      <!-- <inertia ixx="1" ixy="0" ixz="0" iyy="1" iyz="0" izz="1" /> -->
-      <inertia ixx="0.001" ixy="0" ixz="0" iyy="0.001" iyz="0" izz="0.001" />
-   </inertial>
- </link>
-   <link name="caster">
-    <collision name="collision">
-      <!-- <origin xyz="-0.325 0.0 0.05" rpy="0 1.5707 1.5707"/> -->
-      <geometry>
-        <cylinder  length="0.03" radius="0.0725"/>
-      </geometry>
-    </collision>
-    <visual name="visual">
-      <!-- <origin xyz="-0.325 0.0 -0.075" rpy="0 1.5707 1.5707"/> -->
-      <geometry>
-        <cylinder  length="0.03" radius="0.0725"/>
-      </geometry>
-    </visual>
+<robot name="caster" xmlns:xacro="http://www.ros.org/wiki/xacro">
+  <!-- Casters -->
+  <xacro:property name="caster_radius" value="0.05250" /> <!-- in m -->
+  <xacro:property name="caster_mass"   value="1.00" /> <!-- in kg-->
+  <xacro:macro name="caster" params="sub parent transX transY transZ">
+    <!-- sub: l,r 0,1,2,3 etc -->
+    <!-- parent: parent link name -->
+    <!-- transX transY transZ: xyz position -->
+    <link name="caster_${sub}">
+      <visual>
+        <origin xyz="0 0 0" rpy="0 0 0" />
+        <geometry>
+          <sphere radius="${caster_radius}" />
+        </geometry>
+        <material name="Black" />
+      </visual>
+      <collision>
+        <origin xyz="0 0 0" rpy="0 0 0" />
+        <geometry>
+          <sphere radius="${caster_radius}" />
+        </geometry>
+      </collision>
+      <inertial>
+        <mass value="${caster_mass}" />
+        <origin xyz="0 0 0" />
+        <!-- <xacro:sphere_inertia m="${caster_mass}" r="${caster_radius}" /> -->
+        <inertia ixx="0.001" ixy="0.0" ixz="0.0" iyy="0.001" iyz="0.0" izz="0.001"/>
+      </inertial>
     </link>
-  <joint name="caster_support_joint" type="continuous">
-    <axis xyz="0 0 1"/>
-    <parent link="base_link"/>
-    <child link="caster_support"/>
-    <origin xyz="0.15  0.0 -0.075" rpy="0 0 0"/>
-  </joint>
-  <link name="caster_support">
-    <visual name="visual">
-      <geometry>
-        <box size="0.01 0.01 0.01"/>
-      </geometry>
-    </visual>
-    </link>
-  <joint type="continuous" name="caster_joint">
-    <!-- <origin xyz="0 -0.15 0.075" rpy="0 0 0"/> -->
-    <!-- <origin xyz="0 0.0 -0.10" rpy="0 1.5707 1.5707"/> -->
-    <!-- <origin xyz="0 -0.15 -0.05" rpy="1.57 0 0"/> -->
-    <origin xyz="0.0 0.0 0.0" rpy="1.57 0 0"/>
-    <child link="caster"></child>
-    <parent link="caster_support"></parent>
-    <axis xyz="0 0 1"/>
-    <limit effort="100" velocity="100.0"  lower="-5000" upper="5000" />
-  </joint>
-  <link name="left_wheel">
-    <collision name="collision">
-      <!-- <origin xyz="0 0.0 -0.10" rpy="0 1.5707 1.5707"/> -->
-      <geometry>
-         <cylinder  length="0.03" radius="0.0725"/>
-      </geometry>
-    </collision>
-    <visual name="visual">
-      <!-- <origin xyz="0 0.0 -0.10" rpy="0 0 0"/> -->
-      <geometry>
-        <cylinder  length="0.03" radius="0.0725"/>
-      </geometry>
-    </visual>
-    <inertial>
-      <mass value="1" />
-      <origin xyz="0.15 0.15 -0.05" rpy="1.57 0.0 0.0"/>
-      <inertia ixx="0.001" ixy="0" ixz="0" iyy="0.001" iyz="0" izz="0.001" />
-    </inertial>
-  </link>
-  <joint type="continuous" name="left_wheel_joint">
-    <!-- <origin xyz="0 0.15 0.075" rpy="0 0 0"/> -->
-    <origin xyz="-0.15 0.15 -0.05" rpy="1.57 0 0"/>
-    <child link="left_wheel"></child>
-    <parent link="base_link"></parent>
-    <axis xyz="0 0 1"/>
-    <limit effort="100" velocity="100.0"  lower="-5000" upper="5000" />
-  </joint>
-  <!--link name="visual_right_wheel">
-    <visual name="visual">
-      <origin xyz="0 0.0 0" rpy="0 1.5707 1.5707"/>
-      <geometry>
-        <cylinder  length="0.03" radius="0.0725"/>
-      </geometry>
-    </visual>
-  </link>
-  <joint type="fixed" name="visual_right_wheel_joint">
-    <origin xyz="0.15 -0.15 0.075" rpy="0 0 0"/>
-    <child link="visual_right_wheel">visual_right_wheel</child>
-    <parent link="base_link">base_link</parent>
-    <axis xyz="0 1 0"/>
-  </joint-->
-  <link name="right_wheel">
-    <collision name="collision">
-      <!-- <origin xyz="0 0.0 -0.10" rpy="0 1.5707 1.5707"/> -->
-      <!-- <origin xyz="0 0.15 -0.05" rpy="1.57 0 0"/> -->
-      <geometry>
-         <cylinder  length="0.03" radius="0.0725"/>
-      </geometry>
-    </collision>
-    <visual name="visual">
-      <!-- <origin xyz="0 0.0 -0.10" rpy="0 1.5707 1.5707"/> -->
-      <geometry>
-        <cylinder  length="0.03" radius="0.0725"/>
-      </geometry>
-    </visual>
-    <inertial>
-      <mass value="1" />
-      <origin xyz="0 0.0 0"/>
-      <inertia ixx="0.001" ixy="0" ixz="0" iyy="0.001" iyz="0" izz="0.001" />
-    </inertial>
-  </link>
-  <joint type="continuous" name="right_wheel_joint">
-    <!-- <origin xyz="0 -0.15 0.075" rpy="0 0 0"/> -->
-    <!-- <origin xyz="0 0.0 -0.10" rpy="0 1.5707 1.5707"/> -->
-    <origin xyz="-0.15 -0.15 -0.05" rpy="1.57 0 0"/>
-    <child link="right_wheel"></child>
-    <parent link="base_link"></parent>
-    <axis xyz="0 0 1"/>
-    <limit effort="100" velocity="100.0"  lower="-5000" upper="5000" />
-  </joint>
-  <xacro:sensor_hokuyo name="hokuyo" parent="base_link" size="0.05 0.05 0.05">
-    <origin xyz="0.25 0 0.1" rpy="0 0 0"/>
-  </xacro:sensor_hokuyo>
-  <transmission name="tran1">
-    <type>transmission_interface/SimpleTransmission</type>
-    <joint name="left_wheel_joint">
-      <hardwareInterface>VelocityJointInterface</hardwareInterface>
+    <gazebo reference="caster_${sub}">
+      <turnGravityOff>false</turnGravityOff>
+      <material>Gazebo/Black</material>
+      <mu1 value="0.0"/>
+      <mu2 value="0.0"/>
+    </gazebo>
+    <joint name="caster_${sub}_joint" type="fixed">
+      <parent link="${parent}"/>
+      <child link="caster_${sub}"/>
+      <origin xyz="${transX} ${transY} ${transZ}" rpy="0 0 0" />
     </joint>
-    <actuator name="left_motor">
-      <hardwareInterface>VelocityJointInterface</hardwareInterface>
-      <mechanicalReduction>1</mechanicalReduction>
-    </actuator>
-  </transmission>
-  <transmission name="tran2">
-    <type>transmission_interface/SimpleTransmission</type>
-    <joint name="right_wheel_joint">
-      <hardwareInterface>VelocityJointInterface</hardwareInterface>
-    </joint>
-    <actuator name="right_motor">
-      <hardwareInterface>VelocityJointInterface</hardwareInterface>
-      <mechanicalReduction>1</mechanicalReduction>
-    </actuator>
-  </transmission>
+  </xacro:macro>
 </robot>
