Commit message: fix urdf of gamma

File: orne_description/urdf/gamma/orne_gamma.urdf.xacro (robot description, xacro)
@@ -1,5 +1,5 @@
 <?xml version="1.0"?>
 <!-- Revolute-Revolute Manipulator -->
-<robot name="orne_gamma" xmlns:xacro="http://www.ros.org/wiki/xacro">
+<robot name="orne_gamma" xmlns:xacro="http://ros.org/wiki/xacro">
   <!-- Constants for robot dimensions -->
   <xacro:property name="PI" value="3.1415926535897931"/>
@@ -8,4 +8,5 @@
   <xacro:include filename="$(find orne_description)/urdf/gamma/orne_gamma.gazebo"/>
   <xacro:include filename="$(find orne_description)/urdf/sensors/hokuyo.urdf.xacro"/>
+  <xacro:include filename="$(find orne_description)/urdf/gamma/orne_gamma_caster.urdf.xacro"/>
   <!--Base Footprint-->
   <link name="base_footprint" />
@@ -32,5 +33,5 @@
       </geometry>
     </collision>
-     <collision name="collision">
+     <!-- <collision name="collision">
       <origin xyz="0.15 0.0 -0.075" rpy="1.57 0.0 0.0"/>
       <geometry>
@@ -43,5 +44,5 @@
         <cylinder  length="0.03" radius="0.04625"/>
       </geometry>
-    </visual>
+    </visual> -->
     <!-- <inertial>
       <mass value="20" />
@@ -52,5 +53,6 @@
     <mass value="15" />
     <origin xyz="0 0 0" rpy="0 0 0"/>
-    <inertia ixx="1" ixy="0" ixz="0" iyy="1" iyz="0" izz="1" />
+    <!-- <inertia ixx="0.5" ixy="0" ixz="0" iyy="0.5" iyz="0" izz="0.5" /> -->
+    <inertia ixx="0.25925" ixy="0" ixz="0" iyy="0.32216" iyz="0" izz="0.52516" />
     </inertial>
  </link>
@@ -95,4 +97,6 @@
     <collision name="collision">
       <!-- <origin xyz="0 0.0 -0.10" rpy="0 1.5707 1.5707"/> -->
+      <!-- <origin xyz="-0.15 0.15 -0.05" rpy="-1.57 0.0 0.0"/> -->
+      <origin xyz="0.0 0.0 0.0" rpy="0.0 0.0 0.0"/>
       <geometry>
          <cylinder  length="0.03" radius="0.0725"/>
@@ -101,4 +105,6 @@
     <visual name="visual">
       <!-- <origin xyz="0 0.0 -0.10" rpy="0 0 0"/> -->
+      <!-- <origin xyz="-0.15 0.15 -0.05" rpy="-1.57 0.0 0.0"/> -->
+      <origin xyz="0.0 0.0 0.0" rpy="0.0 0.0 0.0"/>
       <geometry>
         <cylinder  length="0.03" radius="0.0725"/>
@@ -107,6 +113,7 @@
     <inertial>
       <mass value="1" />
-      <origin xyz="-0.15 0.15 -0.05" rpy="-1.57 0.0 0.0"/>
-      <inertia ixx="0.1" ixy="0" ixz="0" iyy="0.1" iyz="0" izz="0.1" />
+      <!-- <origin xyz="-0.15 0.15 -0.05" rpy="-1.57 0.0 0.0"/> -->
+      <origin xyz="0.0 0.0 0.0" rpy="0.0 0.0 0.0"/>
+      <inertia ixx="0.001" ixy="0" ixz="0" iyy="0.002" iyz="0" izz="0.001" />
     </inertial>
   </link>
@@ -118,4 +125,5 @@
     <axis xyz="0 0 1"/>
     <limit effort="100" velocity="100.0"  lower="-5000" upper="5000" />
+    <dynamics damping="0.1"/>
   </joint>
   <!--link name="visual_right_wheel">
@@ -135,4 +143,6 @@
   <link name="right_wheel">
     <collision name="collision">
+      <!-- <origin xyz="-0.15 -0.15 -0.05" rpy="-1.57 0.0 0.0"/> -->
+      <origin xyz="0.0 0.0 0.0" rpy="0.0 0.0 0.0"/>
       <!-- <origin xyz="0 0.0 -0.10" rpy="0 1.5707 1.5707"/> -->
       <!-- <origin xyz="0 0.15 -0.05" rpy="1.57 0 0"/> -->
@@ -143,4 +153,6 @@
     <visual name="visual">
       <!-- <origin xyz="0 0.0 -0.10" rpy="0 1.5707 1.5707"/> -->
+      <!-- <origin xyz="-0.15 -0.15 -0.05" rpy="-1.57 0.0 0.0"/> -->
+      <origin xyz="0.0 0.0 0.0" rpy="0.0 0.0 0.0"/>
       <geometry>
         <cylinder  length="0.03" radius="0.0725"/>
@@ -149,6 +161,7 @@
     <inertial>
       <mass value="1" />
-       <origin xyz="-0.15 0.15 -0.05" rpy="-1.57 0.0 0.0"/>
-      <inertia ixx="0.1" ixy="0" ixz="0" iyy="0.1" iyz="0" izz="0.1" />
+      <!-- <origin xyz="-0.15 -0.15 -0.05" rpy="-1.57 0.0 0.0"/> -->
+      <origin xyz="0.0 0.0 0.0" rpy="0.0 0.0 0.0"/>
+      <inertia ixx="0.001" ixy="0" ixz="0" iyy="0.002" iyz="0" izz="0.001" />
     </inertial>
   </link>
@@ -161,8 +174,12 @@
     <axis xyz="0 0 1"/>
     <limit effort="100" velocity="100.0"  lower="-5000" upper="5000" />
+    <dynamics damping="0.1"/>
   </joint>
   <xacro:sensor_hokuyo name="hokuyo" parent="base_link" size="0.05 0.05 0.05">
     <origin xyz="0.25 0 0.1" rpy="0 0 0"/>
   </xacro:sensor_hokuyo>
+  <xacro:caster sub="0" parent="base_link" transX="0.15" transY="0.0" transZ="-0.075" />
+    <!-- <origin xyz="0.25 0 0.1" rpy="0 0 0"/> -->
+  <!-- </xacro:caster> -->
   <transmission name="tran1">
     <type>transmission_interface/SimpleTransmission</type>
@@ -185,3 +202,52 @@
     </actuator>
   </transmission>
+  <joint name="camera_joint" type="fixed">
+    <origin xyz="0.223 -0.011 0.565" rpy="0 0.124 0"/>
+    <parent link="base_link"/>
+    <child link="camera_link"/>
+  </joint>
+  <link name="camera_link">
+    <collision>
+      <origin xyz="0.005 0.011 0.013" rpy="0 0 0"/>
+      <geometry>
+        <box size="0.015 0.030 0.027"/>
+      </geometry>
+    </collision>
+  </link>
+  <joint name="camera_rgb_joint" type="fixed">
+    <origin xyz="0.003 0.011 0.009" rpy="0 0 0"/>
+    <parent link="camera_link"/>
+    <child link="camera_rgb_frame"/>
+  </joint>
+  <link name="camera_rgb_frame"/>
+  <joint name="camera_rgb_optical_joint" type="fixed">
+    <origin xyz="0 0 0" rpy="-1.57 0 -1.57"/>
+    <parent link="camera_rgb_frame"/>
+    <child link="camera_rgb_optical_frame"/>
+  </joint>
+  <link name="camera_rgb_optical_frame"/>
+  <joint name="camera_rgb_left_joint" type="fixed">
+    <origin xyz="0.003 0.111 0.009" rpy="0 0 0.175"/>
+    <parent link="camera_link"/>
+    <child link="camera_rgb_left_frame"/>
+  </joint>
+  <link name="camera_rgb_left_frame"/>
+  <joint name="camera_rgb_optical_left_joint" type="fixed">
+    <origin xyz="0 0 0" rpy="-1.57 0 -1.57"/>
+    <parent link="camera_rgb_left_frame"/>
+    <child link="camera_rgb_optical_left_frame"/>
+  </joint>
+  <link name="camera_rgb_optical_left_frame"/>
+  <joint name="camera_rgb_right_joint" type="fixed">
+    <origin xyz="0.003 -0.089 0.009" rpy="0 0 -0.175"/>
+    <parent link="camera_link"/>
+    <child link="camera_rgb_right_frame"/>
+  </joint>
+  <link name="camera_rgb_right_frame"/>
+  <joint name="camera_rgb_optical_right_joint" type="fixed">
+    <origin xyz="0 0 0" rpy="-1.57 0 -1.57"/>
+    <parent link="camera_rgb_right_frame"/>
+    <child link="camera_rgb_optical_right_frame"/>
+  </joint>
+  <link name="camera_rgb_optical_right_frame"/>
 </robot>

File: orne_description/urdf/gamma/orne_gamma_caster.urdf.xacro (robot description, xacro)
@@ -33,7 +33,8 @@
     </collision>
     <inertial>
-      <mass value="20" />
+      <mass value="10" />
       <origin xyz="-0.08 0 0" rpy="0 0 0"/>
-      <inertia ixx="1" ixy="0" ixz="0" iyy="1" iyz="0" izz="1" />
+      <!-- <inertia ixx="1" ixy="0" ixz="0" iyy="1" iyz="0" izz="1" /> -->
+      <inertia ixx="0.001" ixy="0" ixz="0" iyy="0.001" iyz="0" izz="0.001" />
    </inertial>
  </link>
@@ -42,5 +43,5 @@
       <!-- <origin xyz="-0.325 0.0 0.05" rpy="0 1.5707 1.5707"/> -->
       <geometry>
-        <cylinder  length="0.03" radius="0.04625"/>
+        <cylinder  length="0.03" radius="0.0725"/>
       </geometry>
     </collision>
@@ -48,5 +49,5 @@
       <!-- <origin xyz="-0.325 0.0 -0.075" rpy="0 1.5707 1.5707"/> -->
       <geometry>
-        <cylinder  length="0.03" radius="0.04625"/>
+        <cylinder  length="0.03" radius="0.0725"/>
       </geometry>
     </visual>
@@ -91,5 +92,5 @@
       <mass value="1" />
       <origin xyz="0.15 0.15 -0.05" rpy="1.57 0.0 0.0"/>
-      <inertia ixx="0.1" ixy="0" ixz="0" iyy="0.1" iyz="0" izz="0.1" />
+      <inertia ixx="0.001" ixy="0" ixz="0" iyy="0.001" iyz="0" izz="0.001" />
     </inertial>
   </link>
@@ -133,5 +134,5 @@
       <mass value="1" />
       <origin xyz="0 0.0 0"/>
-      <inertia ixx="0.1" ixy="0" ixz="0" iyy="0.1" iyz="0" izz="0.1" />
+      <inertia ixx="0.001" ixy="0" ixz="0" iyy="0.001" iyz="0" izz="0.001" />
     </inertial>
   </link>

Commit message: Delete unnecessary comments

File: orne_description/urdf/gamma/orne_gamma.urdf.xacro (robot description, xacro)
@@ -19,13 +19,10 @@
   <link name="base_link">
     <visual>
-      <!-- <origin xyz="-0.15 0 0.1" rpy="0 0 0"/> -->
       <origin xyz="0.0 0.0 0.0" rpy="0.0 0.0 0.0"/>>
       <geometry>
 	    <box size=".485 .43 .15"/>
       </geometry>
-      <!-- <material name="orange"/> -->
     </visual>
     <collision name="collision">
-      <!-- <origin xyz="-0.15 0 0.1" rpy="0 0 0"/> -->
       <origin xyz="0.0 0.0 0.0" rpy="0.0 0.0 0.0"/>>
       <geometry>
@@ -33,69 +30,12 @@
       </geometry>
     </collision>
-     <!-- <collision name="collision">
-      <origin xyz="0.15 0.0 -0.075" rpy="1.57 0.0 0.0"/>
-      <geometry>
-        <cylinder  length="0.03" radius="0.04625"/>
-      </geometry>
-    </collision>
-    <visual name="visual">
-      <origin xyz="0.15 0.0 -0.075" rpy="1.57 0.0 0.0"/>
-      <geometry>
-        <cylinder  length="0.03" radius="0.04625"/>
-      </geometry>
-    </visual> -->
-    <!-- <inertial>
-      <mass value="20" />
-      <origin xyz="-0.08 0 0" rpy="0 0 0"/>
-      <inertia ixx="1" ixy="0" ixz="0" iyy="1" iyz="0" izz="1" />
-   </inertial> -->
    <inertial>
     <mass value="15" />
     <origin xyz="0 0 0" rpy="0 0 0"/>
-    <!-- <inertia ixx="0.5" ixy="0" ixz="0" iyy="0.5" iyz="0" izz="0.5" /> -->
     <inertia ixx="0.25925" ixy="0" ixz="0" iyy="0.32216" iyz="0" izz="0.52516" />
     </inertial>
  </link>
-   <!-- <link name="caster"> -->
-    <!-- <collision name="collision">
-      <origin xyz="0.15 0.0 -0.075" rpy="1.57 0.0 0.0"/>
-      <geometry>
-        <cylinder  length="0.03" radius="0.04625"/>
-      </geometry>
-    </collision>
-    <visual name="visual">
-      <origin xyz="-0.325 0.0 -0.075" rpy="0 1.5707 1.5707"/>
-      <geometry>
-        <cylinder  length="0.03" radius="0.04625"/>
-      </geometry>
-    </visual> -->
-    <!-- </link> -->
-  <!-- <joint name="caster_joint" type="continuous">
-    <axis xyz="0 0 1"/>
-    <parent link="base_link"/>
-    <child link="caster"/>
-    <origin xyz="0.15  0.0 -0.075" rpy="1.57 0 0"/>
-  </joint> -->
-  <!-- <link name="caster_support">
-    <visual name="visual">
-      <geometry>
-        <box size="0.01 0.01 0.01"/>
-      </geometry>
-    </visual>
-    </link> -->
-  <!-- <joint type="continuous" name="caster_joint">
-    <origin xyz="0 -0.15 0.075" rpy="0 0 0"/>
-    <origin xyz="0 0.0 -0.10" rpy="0 1.5707 1.5707"/>
-    <origin xyz="0 -0.15 -0.05" rpy="1.57 0 0"/>
-    <origin xyz="0.0 0.0 0.0" rpy="1.57 0 0"/>
-    <child link="caster"></child>
-    <parent link="caster_support"></parent>
-    <axis xyz="0 0 1"/>
-    <limit effort="100" velocity="100.0"  lower="-5000" upper="5000" />
-  </joint> -->
   <link name="left_wheel">
     <collision name="collision">
-      <!-- <origin xyz="0 0.0 -0.10" rpy="0 1.5707 1.5707"/> -->
-      <!-- <origin xyz="-0.15 0.15 -0.05" rpy="-1.57 0.0 0.0"/> -->
       <origin xyz="0.0 0.0 0.0" rpy="0.0 0.0 0.0"/>
       <geometry>
@@ -104,6 +44,4 @@
     </collision>
     <visual name="visual">
-      <!-- <origin xyz="0 0.0 -0.10" rpy="0 0 0"/> -->
-      <!-- <origin xyz="-0.15 0.15 -0.05" rpy="-1.57 0.0 0.0"/> -->
       <origin xyz="0.0 0.0 0.0" rpy="0.0 0.0 0.0"/>
       <geometry>
@@ -113,5 +51,4 @@
     <inertial>
       <mass value="1" />
-      <!-- <origin xyz="-0.15 0.15 -0.05" rpy="-1.57 0.0 0.0"/> -->
       <origin xyz="0.0 0.0 0.0" rpy="0.0 0.0 0.0"/>
       <inertia ixx="0.001" ixy="0" ixz="0" iyy="0.002" iyz="0" izz="0.001" />
@@ -119,5 +56,4 @@
   </link>
   <joint type="continuous" name="left_wheel_joint">
-    <!-- <origin xyz="0 0.15 0.075" rpy="0 0 0"/> -->
     <origin xyz="-0.15 0.15 -0.05" rpy="-1.57 0 0"/>
     <child link="left_wheel"></child>
@@ -127,24 +63,7 @@
     <dynamics damping="0.1"/>
   </joint>
-  <!--link name="visual_right_wheel">
-    <visual name="visual">
-      <origin xyz="0 0.0 0" rpy="0 1.5707 1.5707"/>
-      <geometry>
-        <cylinder  length="0.03" radius="0.0725"/>
-      </geometry>
-    </visual>
-  </link>
-  <joint type="fixed" name="visual_right_wheel_joint">
-    <origin xyz="0.15 -0.15 0.075" rpy="0 0 0"/>
-    <child link="visual_right_wheel">visual_right_wheel</child>
-    <parent link="base_link">base_link</parent>
-    <axis xyz="0 1 0"/>
-  </joint-->
   <link name="right_wheel">
     <collision name="collision">
-      <!-- <origin xyz="-0.15 -0.15 -0.05" rpy="-1.57 0.0 0.0"/> -->
       <origin xyz="0.0 0.0 0.0" rpy="0.0 0.0 0.0"/>
-      <!-- <origin xyz="0 0.0 -0.10" rpy="0 1.5707 1.5707"/> -->
-      <!-- <origin xyz="0 0.15 -0.05" rpy="1.57 0 0"/> -->
       <geometry>
          <cylinder  length="0.03" radius="0.0725"/>
@@ -152,6 +71,4 @@
     </collision>
     <visual name="visual">
-      <!-- <origin xyz="0 0.0 -0.10" rpy="0 1.5707 1.5707"/> -->
-      <!-- <origin xyz="-0.15 -0.15 -0.05" rpy="-1.57 0.0 0.0"/> -->
       <origin xyz="0.0 0.0 0.0" rpy="0.0 0.0 0.0"/>
       <geometry>
@@ -161,5 +78,4 @@
     <inertial>
       <mass value="1" />
-      <!-- <origin xyz="-0.15 -0.15 -0.05" rpy="-1.57 0.0 0.0"/> -->
       <origin xyz="0.0 0.0 0.0" rpy="0.0 0.0 0.0"/>
       <inertia ixx="0.001" ixy="0" ixz="0" iyy="0.002" iyz="0" izz="0.001" />
@@ -167,6 +83,4 @@
   </link>
   <joint type="continuous" name="right_wheel_joint">
-    <!-- <origin xyz="0 -0.15 0.075" rpy="0 0 0"/> -->
-    <!-- <origin xyz="0 0.0 -0.10" rpy="0 1.5707 1.5707"/> -->
     <origin xyz="-0.15 -0.15 -0.05" rpy="-1.57 0 0"/>
     <child link="right_wheel"></child>
@@ -180,6 +94,4 @@
   </xacro:sensor_hokuyo>
   <xacro:caster sub="0" parent="base_link" transX="0.15" transY="0.0" transZ="-0.075" />
-    <!-- <origin xyz="0.25 0 0.1" rpy="0 0 0"/> -->
-  <!-- </xacro:caster> -->
   <transmission name="tran1">
     <type>transmission_interface/SimpleTransmission</type>

File: orne_description/urdf/gamma/orne_gamma_caster.urdf.xacro (robot description, xacro)
@@ -25,5 +25,4 @@
         <mass value="${caster_mass}" />
         <origin xyz="0 0 0" />
-        <!-- <xacro:sphere_inertia m="${caster_mass}" r="${caster_radius}" /> -->
         <inertia ixx="0.001" ixy="0.0" ixz="0.0" iyy="0.001" iyz="0.0" izz="0.001"/>
       </inertial>
